File: motorboard/IMU.sch (KiCad schematic (older format))
At the start: 16 parts

Commit message: nearrrly there
Parts:
- C? (x6): value 0u1 -> 100n
Connections:
- no-connect marks 0 -> 10
Changed lines of the file:
@@
 encoding utf-8
 Sheet 3 3
-Title ""
-Date ""
-Rev ""
-Comp ""
+Title "IMUs"
+Date "2020-02-12"
+Rev "2"
+Comp "Raihaan Usman"
 Comment1 ""
 Comment2 ""
@@
 P 2650 4950
 F 0 "C?" H 2750 4950 50  0000 L CNN
-F 1 "0u1" H 2750 4850 50  0000 L CNN
+F 1 "100n" H 2750 4850 50  0000 L CNN
 F 2 "" H 2650 4950 50  0001 C CNN
 F 3 "~" H 2650 4950 50  0001 C CNN
@@
 P 5050 3600
 F 0 "C?" H 5142 3646 50  0000 L CNN
-F 1 "0u1" H 5142 3555 50  0000 L CNN
+F 1 "100n" H 5142 3555 50  0000 L CNN
 F 2 "" H 5050 3600 50  0001 C CNN
 F 3 "~" H 5050 3600 50  0001 C CNN
@@
 P 5350 3600
 F 0 "C?" H 5442 3646 50  0000 L CNN
-F 1 "0u1" H 5442 3555 50  0000 L CNN
+F 1 "100n" H 5442 3555 50  0000 L CNN
 F 2 "" H 5350 3600 50  0001 C CNN
 F 3 "~" H 5350 3600 50  0001 C CNN
@@
 P 6950 4950
 F 0 "C?" H 7050 4950 50  0000 L CNN
-F 1 "0u1" H 7050 4850 50  0000 L CNN
+F 1 "100n" H 7050 4850 50  0000 L CNN
 F 2 "" H 6950 4950 50  0001 C CNN
 F 3 "~" H 6950 4950 50  0001 C CNN
@@
 P 9350 3600
 F 0 "C?" H 9442 3646 50  0000 L CNN
-F 1 "0u1" H 9442 3555 50  0000 L CNN
+F 1 "100n" H 9442 3555 50  0000 L CNN
 F 2 "" H 9350 3600 50  0001 C CNN
 F 3 "~" H 9350 3600 50  0001 C CNN
@@
 P 9650 3600
 F 0 "C?" H 9742 3646 50  0000 L CNN
-F 1 "0u1" H 9742 3555 50  0000 L CNN
+F 1 "100n" H 9742 3555 50  0000 L CNN
 F 2 "" H 9650 3600 50  0001 C CNN
 F 3 "~" H 9650 3600 50  0001 C CNN
@@
 Text Notes 5050 1900 0    303  ~ 61
 IMUs!!
+NoConn ~ 2950 4300
+NoConn ~ 2950 4400
+NoConn ~ 2950 4500
+NoConn ~ 4350 4100
+NoConn ~ 4350 4000
+NoConn ~ 7250 4500
+NoConn ~ 7250 4400
+NoConn ~ 7250 4300
+NoConn ~ 8650 4100
+NoConn ~ 8650 4000
 $EndSCHEMATC

Commit message: neater
Parts:
- removed C?: 10n, symbol Device:C_Small
- removed C?: 100n, symbol Device:C_Small
- added C?: 10n, symbol Device:C_Small
- added C?: 100n, symbol Device:C_Small
Connections:
- net GND: now also C?.2, C?.2
- net at U?.21 (CAP): now also C?.1
- net at U?.24 (C1): now also C?.1
Other:
- moved on the sheet: C?

Commit message: PCB build started
Parts:
- C13, C14, C15, C16, C17, C18, C19, C20, C21, C22: renamed from C?; footprint (none) -> Capacitor_SMD:C_0603_1608Metric
- R12, R13, R14, R15: renamed from R?; footprint (none) -> Resistor_SMD:R_0603_1608Metric
- gave numbers to parts that had none: 2
Changed lines of the file:
@@
 P 3650 4200
 AR Path="/5E4D83FF" Ref="U?"  Part="1"
-AR Path="/5E4D3AAB/5E4D83FF" Ref="U?"  Part="1"
-F 0 "U?" H 3200 5100 50  0000 C CNN
+AR Path="/5E4D3AAB/5E4D83FF" Ref="U5"  Part="1"
+F 0 "U5" H 3200 5100 50  0000 C CNN
 F 1 "LSM9DS1" H 3300 5000 50  0000 C CNN
 F 2 "Package_LGA:LGA-24L_3x3.5mm_P0.43mm" H 5150 4950 50  0001 C CNN
@@
 	2350 4100 2350 3950
 $Comp
-L Device:R_Small R?
+L Device:R_Small R13
 U 1 1 5E4DAB80
 P 4450 3600
-F 0 "R?" H 4509 3646 50  0000 L CNN
+F 0 "R13" H 4509 3646 50  0000 L CNN
 F 1 "10k" H 4509 3555 50  0000 L CNN
-F 2 "" H 4450 3600 50  0001 C CNN
+F 2 "Resistor_SMD:R_0603_1608Metric" H 4450 3600 50  0001 C CNN
 F 3 "~" H 4450 3600 50  0001 C CNN
 	1    4450 3600
@@
 $EndComp
 $Comp
-L Device:R_Small R?
+L Device:R_Small R12
 U 1 1 5E4DB01F
 P 2350 3850
-F 0 "R?" V 2150 3750 50  0000 L CNN
+F 0 "R12" V 2150 3750 50  0000 L CNN
 F 1 "10k" V 2250 3750 50  0000 L CNN
-F 2 "" H 2350 3850 50  0001 C CNN
+F 2 "Resistor_SMD:R_0603_1608Metric" H 2350 3850 50  0001 C CNN
 F 3 "~" H 2350 3850 50  0001 C CNN
 	1    2350 3850
@@
 $EndComp
 $Comp
-L power:+3V3 #PWR?
+L power:+3V3 #PWR050
 U 1 1 5E4DBA53
 P 4450 3250
-F 0 "#PWR?" H 4450 3100 50  0001 C CNN
+F 0 "#PWR050" H 4450 3100 50  0001 C CNN
 F 1 "+3V3" H 4465 3423 50  0000 C CNN
 F 2 "" H 4450 3250 50  0001 C CNN
@@
 $EndComp
 $Comp
-L power:+3V3 #PWR?
+L power:+3V3 #PWR047
 U 1 1 5E4DBE1F
 P 2350 3650
-F 0 "#PWR?" H 2350 3500 50  0001 C CNN
+F 0 "#PWR047" H 2350 3500 50  0001 C CNN
 F 1 "+3V3" H 2365 3823 50  0000 C CNN
 F 2 "" H 2350 3650 50  0001 C CNN
@@
 	4450 3400 4750 3400
 $Comp
-L Device:C_Small C?
+L Device:C_Small C15
 U 1 1 5E4E1D07
 P 4750 3600
-F 0 "C?" H 4842 3646 50  0000 L CNN
+F 0 "C15" H 4842 3646 50  0000 L CNN
 F 1 "10u" H 4842 3555 50  0000 L CNN
-F 2 "" H 4750 3600 50  0001 C CNN
+F 2 "Capacitor_SMD:C_0603_1608Metric" H 4750 3600 50  0001 C CNN
 F 3 "~" H 4750 3600 50  0001 C CNN
 	1    4750 3600
@@
 	5050 3400 5050 3500
 $Comp
-L Device:C_Small C?
+L Device:C_Small C16
 U 1 1 5E4E34AB
 P 5050 3600
-F 0 "C?" H 5142 3646 50  0000 L CNN
+F 0 "C16" H 5142 3646 50  0000 L CNN
 F 1 "100n" H 5142 3555 50  0000 L CNN
-F 2 "" H 5050 3600 50  0001 C CNN
+F 2 "Capacitor_SMD:C_0603_1608Metric" H 5050 3600 50  0001 C CNN
 F 3 "~" H 5050 3600 50  0001 C CNN
 	1    5050 3600
@@
 	5350 3400 5350 3500
 $Comp
-L Device:C_Small C?
+L Device:C_Small C17
 U 1 1 5E4E3B61
 P 5350 3600
-F 0 "C?" H 5442 3646 50  0000 L CNN
+F 0 "C17" H 5442 3646 50  0000 L CNN
 F 1 "100n" H 5442 3555 50  0000 L CNN
-F 2 "" H 5350 3600 50  0001 C CNN
+F 2 "Capacitor_SMD:C_0603_1608Metric" H 5350 3600 50  0001 C CNN
 F 3 "~" H 5350 3600 50  0001 C CNN
 	1    5350 3600
@@
 	2800 4200 2800 4250
 $Comp
-L power:GND #PWR?
+L power:GND #PWR049
 U 1 1 5E539E5C
 P 2800 4250
-F 0 "#PWR?" H 2800 4000 50  0001 C CNN
+F 0 "#PWR049" H 2800 4000 50  0001 C CNN
 F 1 "GND" H 2805 4077 50  0000 C CNN
 F 2 "" H 2800 4250 50  0001 C CNN
@@
 	4750 3900 4750 4000
 $Comp
-L power:GND #PWR?
+L power:GND #PWR051
 U 1 1 5E53A6ED
 P 4750 4000
-F 0 "#PWR?" H 4750 3750 50  0001 C CNN
+F 0 "#PWR051" H 4750 3750 50  0001 C CNN
 F 1 "GND" H 4755 3827 50  0000 C CNN
 F 2 "" H 4750 4000 50  0001 C CNN
@@
 	6650 4100 6650 3950
 $Comp
-L Device:R_Small R?
+L Device:R_Small R15
 U 1 1 5E54765C
 P 8750 3600
-F 0 "R?" H 8809 3646 50  0000 L CNN
+F 0 "R15" H 8809 3646 50  0000 L CNN
 F 1 "10k" H 8809 3555 50  0000 L CNN
-F 2 "" H 8750 3600 50  0001 C CNN
+F 2 "Resistor_SMD:R_0603_1608Metric" H 8750 3600 50  0001 C CNN
 F 3 "~" H 8750 3600 50  0001 C CNN
 	1    8750 3600
@@
 $EndComp
 $Comp
-L Device:R_Small R?
+L Device:R_Small R14
 U 1 1 5E547662
 P 6650 3850
-F 0 "R?" V 6450 3750 50  0000 L CNN
+F 0 "R14" V 6450 3750 50  0000 L CNN
 F 1 "10k" V 6550 3750 50  0000 L CNN
-F 2 "" H 6650 3850 50  0001 C CNN
+F 2 "Resistor_SMD:R_0603_1608Metric" H 6650 3850 50  0001 C CNN
 F 3 "~" H 6650 3850 50  0001 C CNN
 	1    6650 3850
@@
 $EndComp
 $Comp
-L power:+3V3 #PWR?
+L power:+3V3 #PWR054
 U 1 1 5E547668
 P 8750 3250
-F 0 "#PWR?" H 8750 3100 50  0001 C CNN
+F 0 "#PWR054" H 8750 3100 50  0001 C CNN
 F 1 "+3V3" H 8765 3423 50  0000 C CNN
 F 2 "" H 8750 3250 50  0001 C CNN
@@
 $EndComp
 $Comp
-L power:+3V3 #PWR?
+L power:+3V3 #PWR052
 U 1 1 5E54766E
 P 6650 3650
-F 0 "#PWR?" H 6650 3500 50  0001 C CNN
+F 0 "#PWR052" H 6650 3500 50  0001 C CNN
 F 1 "+3V3" H 6665 3823 50  0000 C CNN
 F 2 "" H 6650 3650 50  0001 C CNN
@@
 	6650 3750 6650 3650
 $Comp
-L Device:C_Small C?
+L Device:C_Small C18
 U 1 1 5E547675
 P 7000 4950
-F 0 "C?" H 6800 5000 50  0000 L CNN
+F 0 "C18" H 6800 5000 50  0000 L CNN
 F 1 "10n" H 6750 4900 50  0000 L CNN
-F 2 "" H 7000 4950 50  0001 C CNN
+F 2 "Capacitor_SMD:C_0603_1608Metric" H 7000 4950 50  0001 C CNN
 F 3 "~" H 7000 4950 50  0001 C CNN
 	1    7000 4950
@@
 $EndComp
 $Comp
-L Device:C_Small C?
+L Device:C_Small C19
 U 1 1 5E54767B
 P 7200 4950
-F 0 "C?" H 7300 4950 50  0000 L CNN
+F 0 "C19" H 7300 4950 50  0000 L CNN
 F 1 "100n" H 7250 4850 50  0000 L CNN
-F 2 "" H 7200 4950 50  0001 C CNN
+F 2 "Capacitor_SMD:C_0603_1608Metric" H 7200 4950 50  0001 C CNN
 F 3 "~" H 7200 4950 50  0001 C CNN
 	1    7200 4950
@@
 	8750 3400 9050 3400
 $Comp
-L Device:C_Small C?
+L Device:C_Small C20
 U 1 1 5E5476A4
 P 9050 3600
-F 0 "C?" H 9142 3646 50  0000 L CNN
+F 0 "C20" H 9142 3646 50  0000 L CNN
 F 1 "10u" H 9142 3555 50  0000 L CNN
-F 2 "" H 9050 3600 50  0001 C CNN
+F 2 "Capacitor_SMD:C_0603_1608Metric" H 9050 3600 50  0001 C CNN
 F 3 "~" H 9050 3600 50  0001 C CNN
 	1    9050 3600
@@
 $EndComp
 $Comp
-L power:GND #PWR?
+L power:GND #PWR055
 U 1 1 5E5476AA
 P 9050 3800
-F 0 "#PWR?" H 9050 3550 50  0001 C CNN
+F 0 "#PWR055" H 9050 3550 50  0001 C CNN
 F 1 "GND" H 9055 3627 50  0000 C CNN
 F 2 "" H 9050 3800 50  0001 C CNN
@@
 	9350 3400 9350 3500
 $Comp
-L Device:C_Small C?
+L Device:C_Small C21
 U 1 1 5E5476B2
 P 9350 3600
-F 0 "C?" H 9442 3646 50  0000 L CNN
+F 0 "C21" H 9442 3646 50  0000 L CNN
 F 1 "100n" H 9442 3555 50  0000 L CNN
-F 2 "" H 9350 3600 50  0001 C CNN
+F 2 "Capacitor_SMD:C_0603_1608Metric" H 9350 3600 50  0001 C CNN
 F 3 "~" H 9350 3600 50  0001 C CNN
 	1    9350 3600
@@
 	9650 3400 9650 3500
 $Comp
-L Device:C_Small C?
+L Device:C_Small C22
 U 1 1 5E5476BA
 P 9650 3600
-F 0 "C?" H 9742 3646 50  0000 L CNN
+F 0 "C22" H 9742 3646 50  0000 L CNN
 F 1 "100n" H 9742 3555 50  0000 L CNN
-F 2 "" H 9650 3600 50  0001 C CNN
+F 2 "Capacitor_SMD:C_0603_1608Metric" H 9650 3600 50  0001 C CNN
 F 3 "~" H 9650 3600 50  0001 C CNN
 	1    9650 3600
@@
 P 7950 4200
 AR Path="/5E547646" Ref="U?"  Part="1"
-AR Path="/5E4D3AAB/5E547646" Ref="U?"  Part="1"
-F 0 "U?" H 7500 5100 50  0000 C CNN
+AR Path="/5E4D3AAB/5E547646" Ref="U6"  Part="1"
+F 0 "U6" H 7500 5100 50  0000 C CNN
 F 1 "LSM9DS1" H 7600 5000 50  0000 C CNN
 F 2 "Package_LGA:LGA-24L_3x3.5mm_P0.43mm" H 9450 4950 50  0001 C CNN
@@
 	7000 5100 7200 5100
 $Comp
-L power:GND #PWR?
+L power:GND #PWR053
 U 1 1 5E547691
 P 7000 5150
-F 0 "#PWR?" H 7000 4900 50  0001 C CNN
+F 0 "#PWR053" H 7000 4900 50  0001 C CNN
 F 1 "GND" H 7005 4977 50  0000 C CNN
 F 2 "" H 7000 5150 50  0001 C CNN
@@
 	8050 5100 8700 5100
 $Comp
-L Device:C_Small C?
+L Device:C_Small C13
 U 1 1 5EA7D439
 P 2700 4950
-F 0 "C?" H 2500 5000 50  0000 L CNN
+F 0 "C13" H 2500 5000 50  0000 L CNN
 F 1 "10n" H 2450 4900 50  0000 L CNN
-F 2 "" H 2700 4950 50  0001 C CNN
+F 2 "Capacitor_SMD:C_0603_1608Metric" H 2700 4950 50  0001 C CNN
 F 3 "~" H 2700 4950 50  0001 C CNN
 	1    2700 4950
@@
 $EndComp
 $Comp
-L Device:C_Small C?
+L Device:C_Small C14
 U 1 1 5EA7D43F
 P 2900 4950
-F 0 "C?" H 3000 4950 50  0000 L CNN
+F 0 "C14" H 3000 4950 50  0000 L CNN
 F 1 "100n" H 2950 4850 50  0000 L CNN
-F 2 "" H 2900 4950 50  0001 C CNN
+F 2 "Capacitor_SMD:C_0603_1608Metric" H 2900 4950 50  0001 C CNN
 F 3 "~" H 2900 4950 50  0001 C CNN
 	1    2900 4950
@@
 	2700 5100 2900 5100
 $Comp
-L power:GND #PWR?
+L power:GND #PWR048
 U 1 1 5EA7D446
 P 2700 5150
-F 0 "#PWR?" H 2700 4900 50  0001 C CNN
+F 0 "#PWR048" H 2700 4900 50  0001 C CNN
 F 1 "GND" H 2705 4977 50  0000 C CNN
 F 2 "" H 2700 5150 50  0001 C CNN
