File: motorboard/motorboard.kicad_pcb (KiCad board)
At the start: 4 copper layers, 34 parts, among them J1 USB_B, J3 Conn_01x02, M1 Motor_DC, Q3 PMV20ENR, U1 CP2102N-A01-GQFN24, U13 TPS2412PW, U2 ATmega328P-AU, U5 TB6612FNG

Commit message: PCB build started
Parts:
- removed C31: 10u, Capacitor_SMD:CP_Elec_4x5.4
- removed M1: Motor_DC, Connector_PinSocket_2.00mm:PinSocket_1x01_P2.00mm_Vertical
- removed R16: 191k, Resistor_SMD:R_0603_1608Metric
- removed R17: 10k, Resistor_SMD:R_0603_1608Metric
- removed R18: 200k, Resistor_SMD:R_0603_1608Metric
- added A1: Pololu_Breakout_A4988, Module:Pololu_Breakout-16_15.2x20.3mm, F.Cu at (121.9, 116.8)
- added C12: 10u, Capacitor_SMD:C_0603_1608Metric, F.Cu at (172.0, 126.0)
- added C13: 10n, Capacitor_SMD:C_0603_1608Metric, F.Cu at (151.0, 118.0)
- added C14: 100n, Capacitor_SMD:C_0603_1608Metric, F.Cu at (144.0, 111.0)
- added C15: 10u, Capacitor_SMD:C_0603_1608Metric, F.Cu at (135.0, 86.0)
- added C16: 100n, Capacitor_SMD:C_0603_1608Metric, F.Cu at (173.0, 130.0)
- added C17: 100n, Capacitor_SMD:C_0603_1608Metric, F.Cu at (140.0, 86.0)
- added C18: 10n, Capacitor_SMD:C_0603_1608Metric, F.Cu at (151.0, 122.0)
- added C19: 100n, Capacitor_SMD:C_0603_1608Metric, F.Cu at (156.0, 122.0)
- added C20: 10u, Capacitor_SMD:C_0603_1608Metric, F.Cu at (172.0, 114.0)
- added C21: 100n, Capacitor_SMD:C_0603_1608Metric, F.Cu at (135.0, 90.0)
- added C22: 100n, Capacitor_SMD:C_0603_1608Metric, F.Cu at (177.0, 126.0)
- added C3: 33p, Capacitor_SMD:C_0603_1608Metric, F.Cu at (153.0, 98.0)
- added D1: POWER LED, Diode_SMD:D_0603_1608Metric_Castellated, F.Cu at (158.0, 132.0)
- added D2: BLINK LED, Diode_SMD:D_0603_1608Metric_Castellated, F.Cu at (178.0, 130.0)
- added D3: D_Schottky, Diode_SMD:D_SOD-123F, F.Cu at (175.0, 100.0)
- added D4: D_Schottky, Diode_SMD:D_SOD-123F, F.Cu at (173.0, 95.0)
- added J2: USB_B, Connector_USB:USB_B_OST_USB-B1HSxx_Horizontal, F.Cu at (180.3, 100.3)
- added J4: LiPo, Connector_PinHeader_2.54mm:PinHeader_1x02_P2.54mm_Vertical, F.Cu at (108.0, 142.2)
- added J5: UART, Connector_PinHeader_2.54mm:PinHeader_1x02_P2.54mm_Vertical, F.Cu at (155.0, 105.0)
- added J6: Encoders, Connector_PinHeader_2.54mm:PinHeader_1x06_P2.54mm_Vertical, F.Cu at (132.1, 78.7)
- added J7: ICSP, Connector_PinHeader_2.54mm:PinHeader_2x03_P2.54mm_Vertical, F.Cu at (127.0, 102.0)
- added J8: Separate LiPo, Connector_PinHeader_2.54mm:PinHeader_1x02_P2.54mm_Vertical, F.Cu at (170.0, 84.0)
- added JP1: MS3, Jumper:SolderJumper-3_P1.3mm_Open_RoundedPad1.0x1.5mm_NumberLabels, F.Cu at (144.0, 129.0)
- added JP2: MS2, Jumper:SolderJumper-3_P1.3mm_Open_RoundedPad1.0x1.5mm_NumberLabels, F.Cu at (129.0, 112.0)
- added JP3: MS1, Jumper:SolderJumper-3_P1.3mm_Open_RoundedPad1.0x1.5mm_NumberLabels, F.Cu at (163.0, 127.0)
- added JP4: Jumper1, Jumper:SolderJumper-2_P1.3mm_Open_RoundedPad1.0x1.5mm, F.Cu at (147.0, 135.0)
- added JP5: Jumper2, Jumper:SolderJumper-2_P1.3mm_Open_RoundedPad1.0x1.5mm, F.Cu at (165.0, 134.0)
- added Q1: PMV20ENR, Package_TO_SOT_SMD:SOT-23, F.Cu at (139.0, 141.0)
- added R10: 470k, Resistor_SMD:R_0603_1608Metric, F.Cu at (153.0, 140.0)
- added R11: 150k, Resistor_SMD:R_0603_1608Metric, F.Cu at (156.0, 136.0)
- added R12: 10k, Resistor_SMD:R_0603_1608Metric, F.Cu at (157.0, 114.0)
- added R13: 10k, Resistor_SMD:R_0603_1608Metric, F.Cu at (158.0, 118.0)
- added R14: 10k, Resistor_SMD:R_0603_1608Metric, F.Cu at (139.0, 111.0)
- added R15: 10k, Resistor_SMD:R_0603_1608Metric, F.Cu at (151.0, 114.0)
- added R3: 4k7, Resistor_SMD:R_0603_1608Metric, F.Cu at (122.0, 108.0)
- added R4: 10K, Resistor_SMD:R_0603_1608Metric, F.Cu at (123.0, 112.0)
- added R5: 10k, Resistor_SMD:R_0603_1608Metric, F.Cu at (148.0, 93.0)
- added R6: 470R, Resistor_SMD:R_0603_1608Metric, F.Cu at (158.0, 140.0)
- added R7: 470R, Resistor_SMD:R_0603_1608Metric, F.Cu at (168.0, 103.0)
- added R8: 10k, Resistor_SMD:R_0603_1608Metric, F.Cu at (161.0, 99.0)
- added R9: 100k, Resistor_SMD:R_0603_1608Metric, F.Cu at (173.0, 138.0)
- added U3: TPS2412PW, Package_SO:TSSOP-8_4.4x3mm_P0.65mm, F.Cu at (123.0, 141.0)
- added U6: LSM9DS1, Package_LGA:LGA-24L_3x3.5mm_P0.43mm, F.Cu at (145.0, 123.0)
- added Y1: 8MHz, Crystal:Crystal_SMD_3225-4Pin_3.2x2.5mm_HandSoldering, F.Cu at (149.0, 105.0)
- C1: value 0u1 -> 10u
- C11: renamed from C29; footprint Capacitor_SMD:CP_Elec_4x5.4 -> Capacitor_SMD:C_0603_1608Metric
- C11: value 100n -> 10u
- C12: renamed from C30; footprint Capacitor_SMD:CP_Elec_4x5.4 -> Capacitor_SMD:C_0603_1608Metric
- C2: value 0u1 -> 47u
- C4: value 10u -> 33p; footprint Capacitor_SMD:CP_Elec_4x5.4 -> Capacitor_SMD:C_0603_1608Metric
- C5: value 10u -> 100n; footprint Capacitor_SMD:CP_Elec_4x5.4 -> Capacitor_SMD:C_0603_1608Metric
- C6: value 4u7 -> 1u
- C7: value 100n -> 2.2n
- C8, C9: value 1u -> 10u
- J1: value USB_B -> Stepper; footprint Connector_USB:USB_B_OST_USB-B1HSxx_Horizontal -> Connector_PinHeader_2.54mm:PinHeader_1x06_P2.54mm_Vertical
- J3: value Conn_01x02 -> DC Motor; footprint Connector_JST:JST_PH_S2B-PH-K_1x02_P2.00mm_Horizontal -> Connector_PinHeader_2.54mm:PinHeader_1x02_P2.54mm_Vertical
- L1: value 10u -> 1u5
- R1: value 22k -> 10k
- R2: value 43k -> 4k7
- U1: value CP2102N-A01-GQFN24 -> TB6612FNG; footprint Package_DFN_QFN:QFN-24-1EP_4x4mm_P0.5mm_EP2.6x2.6mm_ThermalVias -> Package_SO:SSOP-24_5.3x8.2mm_P0.65mm
- U2: value ATmega328P-AU -> ATmega32U4-AU; footprint Package_QFP:TQFP-32_7x7mm_P0.8mm -> Package_QFP:TQFP-44_10x10mm_P0.8mm
- U5: value TB6612FNG -> LSM9DS1; footprint Package_SO:SSOP-24_5.3x8.2mm_P0.65mm -> Package_LGA:LGA-24L_3x3.5mm_P0.43mm
- moved C2 193.6 mm to (115.0, 128.0)
- moved J1 169.0 mm to (108.0, 119.4)
- moved R2 164.3 mm to (134.0, 111.0)
- moved U2 157.3 mm to (138.4, 100.3)
- moved R1 136.1 mm to (166.0, 78.0)
- moved C7 135.6 mm to (116.0, 143.0)
- moved C6 131.2 mm to (129.0, 97.0)
- moved C1 129.8 mm to (172.0, 122.0)
- moved U1 129.0 mm to (162.6, 86.4)
- moved C7 123.6 mm to (146.0, 140.0)
- moved R10 122.1 mm to (150.0, 129.0)
- moved Q1 115.3 mm to (140.0, 135.0)
- moved U3 115.0 mm to (132.0, 141.0)
- moved R9 111.9 mm to (173.0, 142.0)
- moved R11 100.9 mm to (155.0, 128.0)
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- renumbered C28 to C7, D5 to D3, L3 to L1, Q3 to Q1, R23 to R10, R24 to R11, R19 to R8, R21 to R9, U13 to U3
Connections:
- net /power/VO renamed Net-(C10-Pad1)
- C1 pad 1: Net-(C1-Pad1) -> +3V3
- C11 pad 1: Net-(C11-Pad1) -> +3V3
- C2 pad 1: DTR -> GND
- C2 pad 2: Net-(C2-Pad2) -> +15V
- C4 pad 1: VDD -> Net-(C4-Pad1)
- C5 pad 1: VDD -> Net-(C5-Pad1)
- C6 pad 1: +5V -> Net-(C6-Pad1)
- C7 pad 1: Net-(C28-Pad1) -> Net-(C7-Pad1)
- C7 pad 2: +BATT -> +15V
- C7 pad 2: Net-(C7-Pad2) -> +15V
- C8 pad 1: Net-(C8-Pad1) -> VDD
- C9 pad 1: GND -> VDD
- C9 pad 2: +10V -> GND
- J1 pad 1: VBUS -> 1B
- J1 pad 3: Net-(J1-Pad3) -> 1A
- J1 pad 4: GND -> 2A
- J1 pad 5: GND -> Net-(J1-Pad5)
- J3 pad 1: +BATT -> AO1
- J3 pad 2: GND -> AO2
- L1 pad 1: Net-(L3-Pad1) -> Net-(L1-Pad1)
- L1 pad 2: Net-(L3-Pad2) -> Net-(L1-Pad2)
- L1 pad 1: +5V -> Net-(L1-Pad1)
- Q1 pad 2: +BATT -> +15V
- Q1 pad 3: VDD -> Net-(JP4-Pad1)
- R1 pad 1: VBUS -> +3V3
- R2 pad 1: Net-(R1-Pad2) -> +3V3
- R2 pad 2: GND -> SCL
- U1 pad 1: Net-(U1-Pad1) -> AO1
- U1 pad 10: Net-(U1-Pad10) -> GND
- U1 pad 13: Net-(U1-Pad13) -> +10V
- U1 pad 14: Net-(U1-Pad14) -> +10V
- U1 pad 18: Net-(U1-Pad18) -> GND
- U1 pad 19: /RTS -> Net-(R1-Pad2)
- U1 pad 2: GND -> AO1
- U1 pad 20: RX -> +3V3
- U1 pad 21: TX -> AIN1
- U1 pad 22: Net-(U1-Pad22) -> AIN2
- U1 pad 23: DTR -> PWMA
- U1 pad 24: Net-(U1-Pad24) -> +10V
- U1 pad 3: Net-(J1-Pad3) -> GND
- U1 pad 4: Net-(J1-Pad2) -> GND
- U1 pad 5: +3V3 -> AO2
- U1 pad 6: +3V3 -> AO2
- U1 pad 7: VBUS -> Net-(U1-Pad7)
- U1 pad 8: Net-(R1-Pad2) -> Net-(U1-Pad8)
- U1 pad 9: Net-(U1-Pad9) -> GND
- U2 pad 10: Net-(U2-Pad10) -> MOSI
- U2 pad 11: Net-(U2-Pad11) -> MISO
- U2 pad 12: Net-(U2-Pad12) -> PWMB
- U2 pad 13: Net-(U2-Pad13) -> RST
- U2 pad 14: Net-(U2-Pad14) -> +3V3
- U2 pad 15: MOSI -> GND
- U2 pad 16: MISO -> Net-(C4-Pad1)
- U2 pad 17: SCK -> Net-(C3-Pad1)
- U2 pad 18: +3V3 -> SCL
- U2 pad 19: Net-(U2-Pad19) -> SDA
- U2 pad 2: Net-(U2-Pad2) -> +5V
- U2 pad 20: Net-(C1-Pad1) -> RX
- U2 pad 21: GND -> TX
- U2 pad 23: Net-(U2-Pad23) -> GND
- U2 pad 24: Net-(U2-Pad24) -> +3V3
- U2 pad 25: Net-(U2-Pad25) -> AIN2
- U2 pad 29: Net-(C2-Pad2) -> Net-(U2-Pad29)
- U2 pad 3: GND -> D-
- U2 pad 30: RX -> PWMA
- U2 pad 31: TX -> AIN1
- U2 pad 32: Net-(U2-Pad32) -> 13
- U2 pad 4: +3V3 -> D+
- U2 pad 6: +3V3 -> Net-(C6-Pad1)
- U2 pad 7: Net-(U2-Pad7) -> +5V
- U2 pad 9: Net-(U2-Pad9) -> SCK
- U3 pad 1: VDD -> Net-(JP4-Pad1)
- U3 pad 6: VDD -> Net-(JP4-Pad1)
- U3 pad 7: +BATT -> +15V
- U3 pad 8: Net-(C28-Pad1) -> Net-(C7-Pad1)
- U5 pad 1: AO1 -> +3V3
- U5 pad 10: GND -> Net-(U5-Pad10)
- U5 pad 11: BO1 -> Net-(U5-Pad11)
- U5 pad 12: BO1 -> Net-(U5-Pad12)
- U5 pad 13: +10V -> Net-(U5-Pad13)
- U5 pad 14: +10V -> GND
- U5 pad 15: PWMB -> GND
- U5 pad 16: BIN2 -> GND
- U5 pad 17: BIN1 -> GND
- U5 pad 19: Net-(R4-Pad2) -> GND
- U5 pad 2: AO1 -> SCL
- U5 pad 20: +3V3 -> GND
- U5 pad 21: AIN1 -> Net-(C13-Pad1)
- U5 pad 22: AIN2 -> +3V3
- U5 pad 23: PWMA -> +3V3
- U5 pad 24: +10V -> Net-(C14-Pad1)
- U5 pad 3: GND -> +3V3
- U5 pad 4: GND -> SDA
- U5 pad 5: AO2 -> GND
- U5 pad 6: AO2 -> GND
- U5 pad 7: BO2 -> Net-(R12-Pad2)
- U5 pad 8: BO2 -> Net-(R13-Pad2)
- U5 pad 9: GND -> Net-(U5-Pad9)
Other:
- board outline added: 94 x 94 mm
