File: motorboard/motorboard.kicad_pcb (KiCad board)
At the start: 4 copper layers, 94 x 94 mm, 64 parts, among them J1 Stepper, J2 USB_B, J3 DC Motor, J4 LiPo, J5 UART, J6 Encoders, J7 ICSP, J8 Separate LiPo, Q1 PMV20ENR, U1 TB6612FNG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

Commit message: GitHub works again!
Parts:
- moved J2 7.93 mm to (181.6, 105.1)
- moved R7 1.99 mm to (180.3, 88.9), turned to 270 degrees
- moved R6 1.71 mm to (180.3, 101.6), turned to 90 degrees
- moved D1 1.67 mm to (180.3, 97.8), turned to 270 degrees
- moved D2 1.66 mm to (180.3, 94.0), turned to 90 degrees
- moved C17 1.12 mm to (177.0, 71.1)
- turned R12 to 90 degrees
- turned R15 to 180 degrees
Routing:
- net +3V3: track 20.9 -> 128.3 mm, vias 4 -> 7
- net SDA: track 12.9 -> 90.2 mm, vias 0 -> 2
- net D+: track 2.03 -> 62.3 mm, vias 1 -> 2
- net D-: track 1.95 -> 60.6 mm, vias 1 -> 2
- net A2: track 0.00 -> 50.8 mm, vias 0 -> 1
- net A1: track 0.00 -> 45.6 mm, vias 0 -> 1
- net SCK: track 0.00 -> 45.5 mm, vias 0 -> 2
- net 13: track 0.00 -> 43.9 mm, vias 0 -> 2
- net GND: track 31.5 -> 74.1 mm
- net VDD: track 22.5 -> 59.9 mm, vias 0 -> 2
- net RST: track 8.59 -> 45.0 mm
- net MOSI: track 0.00 -> 36.2 mm, vias 0 -> 2
- net TX: track 0.00 -> 34.5 mm
- net AIN2: track 0.00 -> 34.3 mm
- net RX: track 0.00 -> 33.0 mm
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Other:
- outline, holes or cut-outs redrawn

Commit message: PCB nearly done!
Parts:
- J2: value USB_B -> USB_B_Micro; footprint Connector_USB:USB_B_OST_USB-B1HSxx_Horizontal -> Connector_USB:USB_Micro-B_Molex-105017-0001
- moved J2 10.3 mm to (185.5, 95.5), turned to 90 degrees
Connections:
- J2 pad 4: GND -> Net-(J2-Pad4)
Routing:
- net VDD: track 59.9 -> 125.0 mm, vias 2 -> 3
- net GND: track 74.1 -> 136.1 mm, vias 0 -> 1
- net Net-(C18-Pad1): track 0.00 -> 59.8 mm, vias 0 -> 2
- net SDA: track 90.2 -> 33.3 mm
- net Net-(R8-Pad1): track 0.00 -> 31.5 mm
- net +3V3: track 128.3 -> 156.0 mm, vias 7 -> 10
- net /power/FB_3V3: track 4.43 -> 25.6 mm, vias 0 -> 2
- net MS1: track 0.00 -> 18.6 mm
- net Net-(R12-Pad2): track 0.00 -> 17.5 mm, vias 0 -> 2
- net Net-(R14-Pad2): track 0.00 -> 17.0 mm, vias 0 -> 2
- net Net-(R5-Pad1): track 0.00 -> 13.6 mm
- net MS3: track 0.00 -> 10.8 mm
- net D+: track 62.3 -> 54.2 mm
- net VBUS: track 18.8 -> 26.9 mm
- net D-: track 60.6 -> 52.6 mm
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
Commit message: Literally the last few nets...
Parts:
- moved C13 30.0 mm to (166.4, 88.9)
- moved C14 25.4 mm to (171.4, 88.9)
- moved C19 25.1 mm to (168.9, 91.4)
- moved C10 15.9 mm to (151.1, 90.2), turned to 90 degrees
Routing:
- net GND: track 136.1 -> 195.9 mm, vias 1 -> 3
- net Net-(C6-Pad1): track 0.00 -> 44.4 mm
- net Net-(C5-Pad1): track 0.00 -> 40.8 mm
- net Net-(L1-Pad2): track 0.00 -> 17.8 mm, vias 0 -> 2
- net AIN1: track 29.5 -> 45.5 mm, vias 2 -> 3
- net Net-(L1-Pad1): track 0.00 -> 15.8 mm, vias 0 -> 2
- net AIN2: track 34.6 -> 42.3 mm
- net PWMA: track 31.3 -> 38.5 mm
- net Net-(C10-Pad1): track 0.00 -> 3.84 mm
- net +5V: track 7.81 -> 9.81 mm
- net +3V3: track 156.0 -> 157.5 mm, vias 10 -> 11
- net Net-(R12-Pad2): track 17.5 -> 18.5 mm
- net (no net): vias 0 -> 1

Commit message: It broke again
Parts:
- added G***: LOGO, iclr-hw:iclr_logo, F.Cu at (125.7, 133.3)
- added REF**: Yeet, MountingHole:MountingHole_6.4mm_M6_Pad_Via, F.Cu at (177.2, 132.8)
- added REF**: Bye, MountingHole:MountingHole_6.4mm_M6_Pad_Via, F.Cu at (177.2, 62.8)
- added REF**: Hi, MountingHole:MountingHole_6.4mm_M6_Pad_Via, F.Cu at (107.2, 62.8)
- added REF**: A_Hole, MountingHole:MountingHole_6.4mm_M6_Pad_Via, F.Cu at (107.2, 132.8)
- C3, C4: value 33p -> 22p
- Y1: footprint Crystal:Crystal_SMD_3225-4Pin_3.2x2.5mm_HandSoldering -> Crystal:Crystal_HC18-U_Vertical
- moved J5 71.1 mm to (102.9, 86.4)
- moved J7 69.7 mm to (102.9, 76.2), turned to 0 degrees
- moved R4 69.0 mm to (110.0, 78.0)
- moved J8 63.9 mm to (101.6, 118.1), turned to 180 degrees
- moved D4 57.4 mm to (117.0, 121.0), turned to 90 degrees
- moved J2 54.4 mm to (151.1, 53.3), turned to 180 degrees
- moved R6 50.4 mm to (133.0, 119.0)
- moved D1 50.0 mm to (133.0, 114.0)
- moved R15 46.9 mm to (136.0, 124.0)
- moved Q1 40.4 mm to (151.1, 134.6), turned to 180 degrees
- moved R8 39.2 mm to (158.0, 112.0)
- moved C20 38.6 mm to (144.0, 94.0)
- moved U3 37.1 mm to (138.4, 134.6)
- moved Y1 36.2 mm to (121.0, 82.0), turned to 180 degrees
- moved JP4 36.0 mm to (141.0, 140.0)
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Connections:
- U1 pad 13: +10V -> +15V
- U1 pad 14: +10V -> +15V
- U1 pad 24: +10V -> +15V
Routing:
- net +15V: track 43.3 -> 132.1 mm, vias 0 -> 4
- net Net-(C18-Pad1): track 59.8 -> 9.31 mm, vias 2 -> 0
- net Net-(C6-Pad1): track 44.4 -> 4.22 mm
- net VDD: track 125.0 -> 85.1 mm
- net VBUS: track 26.9 -> 66.1 mm, vias 0 -> 2
- net Net-(C5-Pad1): track 40.8 -> 10.1 mm, vias 0 -> 2
- net SCL: track 20.7 -> 47.7 mm, vias 2 -> 3
- net +3V3: track 157.5 -> 131.0 mm, vias 11 -> 15
- net AO2: track 0.00 -> 26.0 mm
- net 13: track 43.9 -> 18.0 mm, vias 2 -> 0
- net D+: track 54.2 -> 29.5 mm
- net AO1: track 0.00 -> 24.0 mm
- net D-: track 52.6 -> 28.7 mm
- net Net-(R8-Pad1): track 31.5 -> 8.27 mm
- net AIN1: track 45.5 -> 23.9 mm, vias 3 -> 0
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Other:
- outline, holes or cut-outs redrawn
- copper layers 4 -> 2

Commit message: ready for fab
Parts:
- added G***: LOGO, command block:command block, B.Cu at (154.9, 94.0)
- added REF**: Axes_Lefthand_Xup, iclr-hw:Axes_Lefthand_Xup, F.Cu at (181.6, 116.8)
- added REF**: Axes_Magnetic_Lefthand_Xdown, iclr-hw:Axes_Magnetic_Lefthand_Xdown, F.Cu at (176.5, 116.8)
- renumbered REF** to BottomLeft, REF** to BottomRight, REF** to TopLeft, REF** to TopRight
Other:
- board text added: "Big Brain"
- board text added: "Designed by Raihaan Usman"
- board text added: "H Bridge"
- board text added: "Important"
- board text added: "MOTORBOARD"
- board text added: "REDSTONE POWERED"
- board text added: "Spare Thing"
- board text added: "Stepper Driver"
- board text added: "THE INCREDIBLE"
- board text added: "Ultra Instinct"

Commit message: neater again!
Parts:
- moved L1 10.2 mm to (156.2, 115.6)
- moved R8 9.78 mm to (148.3, 113.4), turned to 90 degrees
- moved R9 9.77 mm to (148.3, 116.7), turned to 90 degrees
- moved R11 7.28 mm to (152.4, 120.7)
- moved C10 6.15 mm to (149.9, 119.9), turned to 270 degrees
- moved Q1 5.08 mm to (146.1, 134.6), turned to 90 degrees
- moved C7 3.50 mm to (143.5, 139.7), turned to 270 degrees
- moved R10 2.01 mm to (152.4, 119.0), turned to 180 degrees
- turned JP4 to 270 degrees
Routing:
- net +3V3: track 131.0 -> 145.8 mm
- net Net-(L1-Pad1): track 14.5 -> 3.28 mm
- net Net-(L1-Pad2): track 14.4 -> 3.28 mm
- net /power/FB_3V3: track 13.1 -> 3.71 mm
- net GND: track 216.0 -> 223.4 mm, vias 14 -> 9
- net Net-(R9-Pad2): track 10.3 -> 3.18 mm
- net Net-(Q1-Pad1): track 10.8 -> 3.77 mm
- net +15V: track 132.1 -> 135.3 mm
- net VBUS: track 66.1 -> 63.8 mm
- net Net-(C7-Pad1): track 13.4 -> 11.3 mm
- net Net-(JP4-Pad1): track 32.0 -> 31.0 mm, vias 0 -> 2
- net VDD: track 85.1 -> 86.0 mm, vias 3 -> 0
Other:
- net class ower added: clearance 0.127, trace_width 1, via_dia 0.6, via_drill 0.35
- board text removed: "REDSTONE POWERED"

Commit message: noob error fixed
Connections:
- D3 pad 2: VBUS -> +5V
- J2 pad 1: VBUS -> +5V
Routing:
- net +5V: track 5.45 -> 84.2 mm, vias 0 -> 3
- net VBUS: track 63.8 -> 0.00 mm, vias 2 -> 0
Other:
- board text added: "Redstone Powered"

Commit message: tweaks
Routing:
- net AO2: track 26.0 -> 30.5 mm
- net AO1: track 24.0 -> 25.6 mm
Changed lines of the file:
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@@
     (thickness 1.6)
     (drawings 14)
-    (tracks 694)
+    (tracks 692)
     (zones 0)
     (modules 72)
@@
   (segment (start 138.418822 75.661285) (end 138.6394 75.661285) (width 0.2) (layer F.Cu) (net 3))
   (segment (start 140.858342 73.442343) (end 140.858342 73.221767) (width 0.2) (layer F.Cu) (net 3))
+  (via (at 171.45 101.6) (size 0.6) (drill 0.35) (layers F.Cu B.Cu) (net 3))
+  (segment (start 171.45 102.7) (end 171.45 101.6) (width 0.2) (layer F.Cu) (net 3))
+  (segment (start 168.4 105) (end 169.15 105) (width 0.2) (layer F.Cu) (net 3) (status 10))
+  (segment (start 169.15 105) (end 171.45 102.7) (width 0.2) (layer F.Cu) (net 3))
+  (via (at 152.4 68.58) (size 0.6) (drill 0.35) (layers F.Cu B.Cu) (net 3))
+  (segment (start 152.43 68.55) (end 152.43 58.6125) (width 0.2) (layer F.Cu) (net 3))
+  (segment (start 152.4 68.58) (end 152.43 68.55) (width 0.2) (layer F.Cu) (net 3))
+  (segment (start 152.43 54.8025) (end 152.43 59.66) (width 0.2) (layer F.Cu) (net 3) (status 10))
+  (segment (start 171.45 101.6) (end 171.45 92.83) (width 1) (layer B.Cu) (net 3))
+  (segment (start 171.45 92.83) (end 162.28 83.66) (width 1) (layer B.Cu) (net 3))
+  (segment (start 152.4 78.86) (end 152.4 68.58) (width 1) (layer B.Cu) (net 3))
+  (segment (start 157.2 83.66) (end 152.4 78.86) (width 1) (layer B.Cu) (net 3))
+  (segment (start 162.28 83.66) (end 157.2 83.66) (width 1) (layer B.Cu) (net 3))
+  (via (at 143.23 78.58) (size 0.6) (drill 0.35) (layers F.Cu B.Cu) (net 3))
+  (segment (start 152.4 78.86) (end 143.51 78.86) (width 1) (layer B.Cu) (net 3))
+  (segment (start 143.51 78.86) (end 143.23 78.58) (width 1) (layer B.Cu) (net 3))
+  (segment (start 139.758186 75.108186) (end 139.758186 75.108185) (width 1) (layer F.Cu) (net 3))
+  (segment (start 138.418822 75.661285) (end 139.205087 75.661285) (width 0.2) (layer F.Cu) (net 3))
+  (segment (start 139.205087 75.661285) (end 139.758186 75.108186) (width 0.2) (layer F.Cu) (net 3))
+  (segment (start 138.032714 75.275177) (end 138.418822 75.661285) (width 0.2) (layer F.Cu) (net 3))
+  (segment (start 137.643806 75.275177) (end 138.032714 75.275177) (width 0.2) (layer F.Cu) (net 3))
+  (segment (start 140.858342 74.00803) (end 139.758186 75.108186) (width 0.2) (layer F.Cu) (net 3))
+  (segment (start 140.472233 72.835658) (end 140.858342 73.221767) (width 0.2) (layer F.Cu) (net 3))
+  (segment (start 140.858342 73.221767) (end 140.858342 74.00803) (width 0.2) (layer F.Cu) (net 3))
+  (segment (start 140.472233 72.44675) (end 140.472233 72.835658) (width 0.2) (layer F.Cu) (net 3))
+  (segment (start 143.23 78.58) (end 139.758186 75.108186) (width 0.2) (layer F.Cu) (net 3))
   (segment (start 139.364008 133.645) (end 138.409504 134.599504) (width 0.2) (layer F.Cu) (net 4))
   (segment (start 141.38 133.645) (end 139.364008 133.645) (width 0.2) (layer F.Cu) (net 4))
@@
   (segment (start 141.2125 126) (end 141.2125 126.475) (width 0.2) (layer F.Cu) (net 5))
   (segment (start 141.2125 126.475) (end 141.43951 126.70201) (width 0.2) (layer F.Cu) (net 5))
-  (via (at 171.45 101.6) (size 0.6) (drill 0.35) (layers F.Cu B.Cu) (net 3))
-  (segment (start 171.45 102.7) (end 171.45 101.6) (width 0.2) (layer F.Cu) (net 3))
-  (segment (start 168.4 105) (end 169.15 105) (width 0.2) (layer F.Cu) (net 3) (status 10))
-  (segment (start 169.15 105) (end 171.45 102.7) (width 0.2) (layer F.Cu) (net 3))
-  (via (at 152.4 68.58) (size 0.6) (drill 0.35) (layers F.Cu B.Cu) (net 3))
-  (segment (start 152.43 68.55) (end 152.43 58.6125) (width 0.2) (layer F.Cu) (net 3))
-  (segment (start 152.4 68.58) (end 152.43 68.55) (width 0.2) (layer F.Cu) (net 3))
-  (segment (start 152.43 54.8025) (end 152.43 59.66) (width 0.2) (layer F.Cu) (net 3) (status 10))
-  (segment (start 171.45 101.6) (end 171.45 92.83) (width 1) (layer B.Cu) (net 3))
-  (segment (start 171.45 92.83) (end 162.28 83.66) (width 1) (layer B.Cu) (net 3))
-  (segment (start 152.4 78.86) (end 152.4 68.58) (width 1) (layer B.Cu) (net 3))
-  (segment (start 157.2 83.66) (end 152.4 78.86) (width 1) (layer B.Cu) (net 3))
-  (segment (start 162.28 83.66) (end 157.2 83.66) (width 1) (layer B.Cu) (net 3))
-  (via (at 143.23 78.58) (size 0.6) (drill 0.35) (layers F.Cu B.Cu) (net 3))
-  (segment (start 152.4 78.86) (end 143.51 78.86) (width 1) (layer B.Cu) (net 3))
-  (segment (start 143.51 78.86) (end 143.23 78.58) (width 1) (layer B.Cu) (net 3))
-  (segment (start 139.758186 75.108186) (end 139.758186 75.108185) (width 1) (layer F.Cu) (net 3))
-  (segment (start 138.418822 75.661285) (end 139.205087 75.661285) (width 0.2) (layer F.Cu) (net 3))
-  (segment (start 139.205087 75.661285) (end 139.758186 75.108186) (width 0.2) (layer F.Cu) (net 3))
-  (segment (start 138.032714 75.275177) (end 138.418822 75.661285) (width 0.2) (layer F.Cu) (net 3))
-  (segment (start 137.643806 75.275177) (end 138.032714 75.275177) (width 0.2) (layer F.Cu) (net 3))
-  (segment (start 140.858342 74.00803) (end 139.758186 75.108186) (width 0.2) (layer F.Cu) (net 3))
-  (segment (start 140.472233 72.835658) (end 140.858342 73.221767) (width 0.2) (layer F.Cu) (net 3))
-  (segment (start 140.858342 73.221767) (end 140.858342 74.00803) (width 0.2) (layer F.Cu) (net 3))
-  (segment (start 140.472233 72.44675) (end 140.472233 72.835658) (width 0.2) (layer F.Cu) (net 3))
-  (segment (start 143.23 78.58) (end 139.758186 75.108186) (width 0.2) (layer F.Cu) (net 3))
   (segment (start 153.775 114.47) (end 153.175 115.07) (width 0.2) (layer F.Cu) (net 7))
   (segment (start 156.21 114.47) (end 153.775 114.47) (width 0.2) (layer F.Cu) (net 7))
@@
   (segment (start 157.69 98.145) (end 153.252098 98.145) (width 0.2) (layer F.Cu) (net 28) (status 10))
   (segment (start 153.252098 98.145) (end 152.54799 97.440892) (width 0.2) (layer F.Cu) (net 28))
-  (segment (start 184.15 90.362999) (end 184.15 88.9) (width 0.2) (layer F.Cu) (net 30) (status 20))
-  (segment (start 183.118399 90.362999) (end 184.15 90.362999) (width 0.2) (layer F.Cu) (net 30))
-  (segment (start 168.394552 96.34799) (end 168.65201 96.605448) (width 0.2) (layer F.Cu) (net 30))
-  (segment (start 164.89 96.845) (end 167.34799 96.845) (width 0.2) (layer F.Cu) (net 30) (status 10))
-  (segment (start 167.34799 96.605448) (end 167.605448 96.34799) (width 0.2) (layer F.Cu) (net 30))
-  (segment (start 178.745 96.845) (end 183.095699 92.494301) (width 0.2) (layer F.Cu) (net 30))
-  (segment (start 183.072999 90.408399) (end 183.118399 90.362999) (width 0.2) (layer F.Cu) (net 30))
-  (segment (start 167.34799 96.845) (end 167.34799 96.605448) (width 0.2) (layer F.Cu) (net 30))
-  (segment (start 168.65201 96.605448) (end 168.65201 96.845) (width 0.2) (layer F.Cu) (net 30))
-  (segment (start 168.65201 96.845) (end 178.745 96.845) (width 0.2) (layer F.Cu) (net 30))
-  (segment (start 183.095699 92.494301) (end 183.072999 92.471601) (width 0.2) (layer F.Cu) (net 30))
-  (segment (start 167.605448 96.34799) (end 168.394552 96.34799) (width 0.2) (layer F.Cu) (net 30))
-  (segment (start 183.072999 92.471601) (end 183.072999 90.408399) (width 0.2) (layer F.Cu) (net 30))
-  (segment (start 164.89 97.495) (end 164.89 96.845) (width 0.2) (layer F.Cu) (net 30) (status 30))
-  (segment (start 176.98799 99.65201) (end 184.15 92.49) (width 0.2) (layer F.Cu) (net 31))
-  (segment (start 166.17201 99.65201) (end 176.98799 99.65201) (width 0.2) (layer F.Cu) (net 31))
+  (segment (start 182.947919 88.9) (end 181.33 90.517919) (width 1) (layer F.Cu) (net 30))
+  (segment (start 184.15 88.9) (end 182.947919 88.9) (width 1) (layer F.Cu) (net 30))
+  (segment (start 181.33 90.517919) (end 181.33 92.55) (width 1) (layer F.Cu) (net 30))
+  (segment (start 181.33 92.55) (end 178.79 95.09) (width 1) (layer F.Cu) (net 30))
+  (segment (start 178.79 95.09) (end 168.63 95.09) (width 1) (layer F.Cu) (net 30))
+  (segment (start 168.37 95.09) (end 168.63 95.09) (width 0.2) (layer F.Cu) (net 30))
+  (segment (start 164.89 97.495) (end 165.965 97.495) (width 0.2) (layer F.Cu) (net 30))
+  (segment (start 167.72 95.09) (end 168.63 95.09) (width 0.2) (layer F.Cu) (net 30))
+  (segment (start 165.965 96.845) (end 167.72 95.09) (width 0.2) (layer F.Cu) (net 30))
+  (segment (start 164.89 96.845) (end 165.965 96.845) (width 0.2) (layer F.Cu) (net 30))
+  (segment (start 166.225 97.495) (end 164.89 97.495) (width 0.2) (layer F.Cu) (net 30))
+  (segment (start 168.63 95.09) (end 166.225 97.495) (width 0.2) (layer F.Cu) (net 30))
+  (segment (start 164.89 97.495) (end 164.89 96.845) (width 0.2) (layer F.Cu) (net 30))
   (segment (start 184.15 92.49) (end 184.15 91.44) (width 0.2) (layer F.Cu) (net 31) (status 20))
-  (segment (start 165.965 99.445) (end 166.17201 99.65201) (width 0.2) (layer F.Cu) (net 31))
-  (segment (start 164.89 99.445) (end 165.965 99.445) (width 0.2) (layer F.Cu) (net 31) (status 10))
   (segment (start 164.89 100.095) (end 164.89 99.445) (width 0.2) (layer F.Cu) (net 31) (status 30))
+  (segment (start 177.345 100.095) (end 184.15 93.29) (width 1) (layer F.Cu) (net 31))
+  (segment (start 184.15 93.29) (end 184.15 91.44) (width 1) (layer F.Cu) (net 31))
+  (segment (start 164.89 100.095) (end 177.345 100.095) (width 1) (layer F.Cu) (net 31))
   (segment (start 115.57 113.6925) (end 115.57 107.95) (width 1) (layer F.Cu) (net 33) (status 20))
   (segment (start 139.62299 134.69701) (end 140.025 134.295) (width 0.2) (layer F.Cu) (net 33))
