File: motorboard/_autosave-power.sch (KiCad schematic (older format))
At the start: 19 parts, among them J8 Separate LiPo, Q1 PMV20ENR, U3 TPS2412PW, U4 TPS63070

Commit message: Sad day for GitHub
Parts:
- U4: footprint iclr-fp:Texas_PowerVFQFN_15 -> main:Texas_PowerVFQFN_15
Changed lines of the file:
@@
 F 0 "U4" H 6950 4716 50  0000 C CNN
 F 1 "TPS63070" H 6950 4625 50  0000 C CNN
-F 2 "iclr-fp:Texas_PowerVFQFN_15" H 6800 4050 50  0001 L BNN
+F 2 "main:Texas_PowerVFQFN_15" H 6800 4050 50  0001 L BNN
 F 3 "TPS63070RNMT" H 6950 4050 50  0001 L BNN
 F 4 "https://www.digikey.com/product-detail/en/texas-instruments/TPS63070RNMT/296-44764-1-ND/6193751?utm_source=snapeda&utm_medium=aggregator&utm_campaign=symbol" H 6800 4050 50  0001 L BNN "Field4"
