File: motorboard/motorboard.sch (KiCad schematic (older format))
At the start: 15 parts, among them J1 USB_B, SW1 SW_Push, U1 CP2102N-A01-GQFN24, U2 ATmega328P-AU

Commit message: Replaced ATMega328
Parts:
- removed C2: 0u1, Capacitor_SMD:C_0603_1608Metric, symbol Device:C_Small
- removed SW1: SW_Push, symbol Switch:SW_Push
- removed U2: ATmega328P-AU, Package_QFP:TQFP-32_7x7mm_P0.8mm, symbol MCU_Microchip_ATmega:ATmega328P-AU
- added C?: 1u, Capacitor_SMD:C_0603_1608Metric, symbol Device:C_Small
- added J?: USB_B, Connector_USB:USB_B_OST_USB-B1HSxx_Horizontal, symbol Connector:USB_B
- added R? (x2): 10k, symbol Device:R_Small
- added R?: 4k7, symbol Device:R_Small
- added U?: ATmega32U4-AU, Package_QFP:TQFP-44_10x10mm_P0.8mm, symbol MCU_Microchip_ATmega:ATmega32U4-AU
Connections:
- net labels added: D+, D-, DIR, PGO
- net labels removed: IMU1, IMU2
- wire segments 96 -> 99
Other:
- note added: "ATMega32u4-AU"
- note added: "I2C Pullup"
- note removed: "ATMega328P-AU"
- moved on the sheet: C1, C?, J1, R1, R2, R3, U1

Commit message: update 09/02
Parts:
- added U?: LSM9DS1, Package_LGA:LGA-24L_3x3.5mm_P0.43mm, symbol Sensor_Motion:LSM9DS1
Other:
- moved on the sheet: C1, C?, J?, R3, R?, U?

Commit message: Complete - Rev1
Parts:
- removed C?: 100n, symbol Device:C_Small
- removed J1: USB_B, Connector_USB:USB_B_OST_USB-B1HSxx_Horizontal, symbol Connector:USB_B
- removed R1: 22k, Resistor_SMD:R_0603_1608Metric, symbol Device:R
- removed R2: 43k, Resistor_SMD:R_0603_1608Metric, symbol Device:R
- removed R?: 4k7, symbol Device:R_Small
- removed U1: CP2102N-A01-GQFN24, Package_DFN_QFN:QFN-24-1EP_4x4mm_P0.5mm_EP2.6x2.6mm_ThermalVias, symbol Interface_USB:CP2102N-A01-GQFN24
- removed U?: AS5600-ASOM, SOIC127P600X175-8N, symbol AS5600:AS5600-ASOM
- removed U?: LSM9DS1, Package_LGA:LGA-24L_3x3.5mm_P0.43mm, symbol Sensor_Motion:LSM9DS1
- added A?: Pololu_Breakout_A4988, Module:Pololu_Breakout-16_15.2x20.3mm, symbol Driver_Motor:Pololu_Breakout_A4988
- added C?: 47u, symbol Device:C_Small
- added C? (x2): 33p, symbol Device:C_Small
- added J?: Encoders, symbol Connector:Conn_01x05_Male
- added J?: ICSP, symbol Connector_Generic:Conn_02x03_Odd_Even
- added J?: UART, symbol Connector:Conn_01x02_Male
- added J?: LiPo, Connector_JST:JST_PH_S2B-PH-K_1x02_P2.00mm_Horizontal, symbol Connector_Generic:Conn_01x02
- added R?: 10k, symbol Device:R_Small
- added Y?: 8MHz, symbol Device:Crystal
- J?: value Conn_01x04_Male -> Stepper
Connections:
- net labels added: +15V, +5V, 1A, 1B, 2A, 2B, A1, A2, RST, STEP
- net labels removed: BIN1, BIN2, DTR, ENC, PGO, RTS
- wire segments 99 -> 116
- no-connect marks 11 -> 0
Other:
- note added: "Black"
- note added: "Connectors"
- note added: "Encoders"
- note added: "Green"
- note added: "Stepper Driver"
- note added: "USB & LiPo"
- note removed: "Encoder"
- note removed: "USB Interface"
- note removed: "USB to UART"
- moved on the sheet: C1, C?, J?, R3, R?, U?

Commit message: nearrrly there
Parts:
- removed J?: Encoders, symbol Connector:Conn_01x05_Male
- added D?: POWER LED, Diode_SMD:D_0603_1608Metric_Pad1.05x0.95mm_HandSolder, symbol Device:LED_Small
- added D?: BLINK LED, Diode_SMD:D_0603_1608Metric_Pad1.05x0.95mm_HandSolder, symbol Device:LED_Small
- added J?: Encoders, symbol Connector:Conn_01x06_Male
- added J?: DC Motor, symbol Connector:Conn_01x02_Male
- added JP? (x3): Jumper, symbol Jumper:SolderJumper_3_Open
- added R? (x2): 470R, symbol Device:R_Small
- C1: value 0u1 -> 100n
- R? (x2): value 10k -> 4k7
Connections:
- net labels added: 13, MS1, MS2, MS3
- net labels removed: BO1, BO2
- wire segments 116 -> 130
- no-connect marks 0 -> 18
Other:
- note added: "Motor Interface"
- note removed: "Stepper Motor"
- note removed: "White"
- note removed: "Yellow"
- moved on the sheet: A?, C1, C?, J?, R3, R?, U?, Y?

Commit message: tidying things
Parts:
- removed JP? (x3): Jumper, symbol Jumper:SolderJumper_3_Open
- added JP?: MS1, symbol Jumper:SolderJumper_3_Open
- added JP?: MS3, symbol Jumper:SolderJumper_3_Open
- added JP?: MS2, symbol Jumper:SolderJumper_3_Open
Connections:
- wire segments 130 -> 141
Changed lines of the file:
@@
 Text Notes 5800 3000 0    50   ~ 0
 Red
-$Comp
-L power:+3V3 #PWR?
-U 1 1 5E52FFC7
-P 6450 2350
-F 0 "#PWR?" H 6450 2200 50  0001 C CNN
-F 1 "+3V3" H 6350 2500 50  0000 C CNN
-F 2 "" H 6450 2350 50  0001 C CNN
-F 3 "" H 6450 2350 50  0001 C CNN
-	1    6450 2350
-	1    0    0    -1
-$EndComp
 Wire Wire Line
 	4500 2450 4400 2450
@@
 Text Notes 4000 6000 0    207  ~ 0
 Connectors
-$Comp
-L Device:Crystal Y?
-U 1 1 5E5C2710
-P 8450 1650
-F 0 "Y?" V 8450 1500 50  0000 R CNN
-F 1 "8MHz" V 8650 1750 50  0000 R CNN
-F 2 "" H 8450 1650 50  0001 C CNN
-F 3 "~" H 8450 1650 50  0001 C CNN
-	1    8450 1650
-	0    -1   -1   0
-$EndComp
 Wire Wire Line
 	8700 1550 8650 1550
@@
 	8650 1550 8650 1500
 Wire Wire Line
-	8650 1500 8450 1500
-Wire Wire Line
 	8700 1750 8650 1750
 Wire Wire Line
 	8650 1750 8650 1800
-Wire Wire Line
-	8650 1800 8450 1800
 $Comp
 L power:GND #PWR?
@@
 	0    1    1    0
 $EndComp
-Wire Wire Line
-	8450 1500 8300 1500
-Connection ~ 8450 1500
-Wire Wire Line
-	8450 1800 8300 1800
-Connection ~ 8450 1800
 Wire Wire Line
 	8100 1800 8050 1800
@@
 	1    0    0    -1
 $EndComp
-$Comp
-L Jumper:SolderJumper_3_Open JP?
-U 1 1 5E72A5E4
-P 7250 2650
-F 0 "JP?" V 7100 2700 50  0000 L CNN
-F 1 "Jumper" H 7150 2750 50  0000 L CNN
-F 2 "" H 7250 2650 50  0001 C CNN
-F 3 "~" H 7250 2650 50  0001 C CNN
-	1    7250 2650
-	0    -1   -1   0
-$EndComp
-$Comp
-L Jumper:SolderJumper_3_Open JP?
-U 1 1 5E72EB25
-P 6450 2650
-F 0 "JP?" V 6300 2700 50  0000 L CNN
-F 1 "Jumper" H 6350 2750 50  0000 L CNN
-F 2 "" H 6450 2650 50  0001 C CNN
-F 3 "~" H 6450 2650 50  0001 C CNN
-	1    6450 2650
-	0    -1   -1   0
-$EndComp
 Text GLabel 4500 3050 0    50   Input ~ 0
 MS1
@@
 Text GLabel 4500 3250 0    50   Input ~ 0
 MS3
-$Comp
-L Jumper:SolderJumper_3_Open JP?
-U 1 1 5E736A16
-P 6850 3050
-F 0 "JP?" V 6700 3100 50  0000 L CNN
-F 1 "Jumper" H 6750 3150 50  0000 L CNN
-F 2 "" H 6850 3050 50  0001 C CNN
-F 3 "~" H 6850 3050 50  0001 C CNN
-	1    6850 3050
-	0    -1   -1   0
-$EndComp
-Text GLabel 7000 3050 2    50   Input ~ 0
-MS1
-Text GLabel 7400 2650 2    50   Input ~ 0
-MS2
-Text GLabel 6600 2650 2    50   Input ~ 0
-MS3
-Connection ~ 6850 2450
-Wire Wire Line
-	6850 2850 6850 2450
 $Comp
 L power:+3V3 #PWR?
@@
 Wire Wire Line
 	10850 2400 10850 2300
-Wire Wire Line
-	6450 2450 6850 2450
-Wire Wire Line
-	6850 2450 7250 2450
-$Comp
-L power:GND #PWR?
-U 1 1 5E7A289F
-P 6450 2850
-F 0 "#PWR?" H 6450 2600 50  0001 C CNN
-F 1 "GND" H 6600 2750 50  0000 C CNN
-F 2 "" H 6450 2850 50  0001 C CNN
-F 3 "" H 6450 2850 50  0001 C CNN
-	1    6450 2850
-	1    0    0    -1
-$EndComp
-$Comp
-L power:GND #PWR?
-U 1 1 5E7A3015
-P 6850 3200
-F 0 "#PWR?" H 6850 2950 50  0001 C CNN
-F 1 "GND" H 7000 3100 50  0000 C CNN
-F 2 "" H 6850 3200 50  0001 C CNN
-F 3 "" H 6850 3200 50  0001 C CNN
-	1    6850 3200
-	1    0    0    -1
-$EndComp
-$Comp
-L power:GND #PWR?
-U 1 1 5E7A32E6
-P 7250 2850
-F 0 "#PWR?" H 7250 2600 50  0001 C CNN
-F 1 "GND" H 7400 2750 50  0000 C CNN
-F 2 "" H 7250 2850 50  0001 C CNN
-F 3 "" H 7250 2850 50  0001 C CNN
-	1    7250 2850
-	1    0    0    -1
-$EndComp
 Wire Wire Line
 	9900 2350 10100 2350
@@
 Wire Wire Line
 	8500 2650 8700 2650
-Wire Wire Line
-	6450 2450 6450 2350
-Connection ~ 6450 2450
+$Comp
+L power:GND #PWR?
+U 1 1 5E8ED772
+P 7250 3200
+F 0 "#PWR?" H 7250 2950 50  0001 C CNN
+F 1 "GND" H 7400 3100 50  0000 C CNN
+F 2 "" H 7250 3200 50  0001 C CNN
+F 3 "" H 7250 3200 50  0001 C CNN
+	1    7250 3200
+	1    0    0    -1
+$EndComp
+Text GLabel 6950 2350 2    50   Input ~ 0
+MS3
+Text GLabel 6950 2950 2    50   Input ~ 0
+MS2
+Text GLabel 6950 3250 2    50   Input ~ 0
+MS1
+$Comp
+L Jumper:SolderJumper_3_Open JP?
+U 1 1 5E8ED785
+P 6850 2500
+F 0 "JP?" H 6600 2600 50  0000 L CNN
+F 1 "MS3" H 6900 2400 50  0000 L CNN
+F 2 "" H 6850 2500 50  0001 C CNN
+F 3 "~" H 6850 2500 50  0001 C CNN
+	1    6850 2500
+	-1   0    0    1
+$EndComp
+$Comp
+L Jumper:SolderJumper_3_Open JP?
+U 1 1 5E8ED78B
+P 6850 2800
+F 0 "JP?" H 6600 2850 50  0000 L CNN
+F 1 "MS2" H 6900 2900 50  0000 L CNN
+F 2 "" H 6850 2800 50  0001 C CNN
+F 3 "~" H 6850 2800 50  0001 C CNN
+	1    6850 2800
+	-1   0    0    -1
+$EndComp
+$Comp
+L power:+3V3 #PWR?
+U 1 1 5E8ED791
+P 6450 2400
+F 0 "#PWR?" H 6450 2250 50  0001 C CNN
+F 1 "+3V3" H 6350 2550 50  0000 C CNN
+F 2 "" H 6450 2400 50  0001 C CNN
+F 3 "" H 6450 2400 50  0001 C CNN
+	1    6450 2400
+	1    0    0    -1
+$EndComp
+$Comp
+L Jumper:SolderJumper_3_Open JP?
+U 1 1 5E8ED77F
+P 6850 3100
+F 0 "JP?" H 6650 3000 50  0000 L CNN
+F 1 "MS1" H 6650 3200 50  0000 L CNN
+F 2 "" H 6850 3100 50  0001 C CNN
+F 3 "~" H 6850 3100 50  0001 C CNN
+	1    6850 3100
+	1    0    0    -1
+$EndComp
+Wire Wire Line
+	7050 3100 7250 3100
+Wire Wire Line
+	7250 3100 7250 3200
+Wire Wire Line
+	7050 2500 7250 2500
+Wire Wire Line
+	7250 2800 7250 3100
+Wire Wire Line
+	7050 2800 7250 2800
+Connection ~ 7250 3100
+Wire Wire Line
+	7250 2800 7250 2500
+Connection ~ 7250 2800
+Wire Wire Line
+	6950 3250 6850 3250
+Wire Wire Line
+	6950 2950 6850 2950
+Wire Wire Line
+	6950 2350 6850 2350
+Wire Wire Line
+	6450 2500 6650 2500
+Wire Wire Line
+	6650 3100 6450 3100
+Connection ~ 6450 2500
+Wire Wire Line
+	6650 2800 6450 2800
+Wire Wire Line
+	6450 2500 6450 2800
+Connection ~ 6450 2800
+Wire Wire Line
+	6450 2800 6450 3100
+Wire Wire Line
+	6450 2400 6450 2500
+Connection ~ 8450 1800
+Connection ~ 8450 1500
+Wire Wire Line
+	8450 1800 8300 1800
+Wire Wire Line
+	8650 1800 8450 1800
+Wire Wire Line
+	8450 1500 8300 1500
+Wire Wire Line
+	8650 1500 8450 1500
+$Comp
+L Device:Crystal Y?
+U 1 1 5E5C2710
+P 8450 1650
+F 0 "Y?" V 8450 1500 50  0000 R CNN
+F 1 "8MHz" V 8650 1750 50  0000 R CNN
+F 2 "" H 8450 1650 50  0001 C CNN
+F 3 "~" H 8450 1650 50  0001 C CNN
+	1    8450 1650
+	0    -1   -1   0
+$EndComp
 $EndSCHEMATC

Commit message: Debugged
*Should* work
Changed lines of the file:
@@
 $EndComp
-Wire Wire Line
-	8700 1150 8700 1250
 Wire Wire Line
 	9900 2950 10100 2950
@@
 L power:+3V3 #PWR?
 U 1 1 5E486812
-P 5700 6600
-F 0 "#PWR?" H 5700 6450 50  0001 C CNN
-F 1 "+3V3" H 5715 6773 50  0000 C CNN
-F 2 "" H 5700 6600 50  0001 C CNN
-F 3 "" H 5700 6600 50  0001 C CNN
-	1    5700 6600
+P 5750 6600
+F 0 "#PWR?" H 5750 6450 50  0001 C CNN
+F 1 "+3V3" H 5765 6773 50  0000 C CNN
+F 2 "" H 5750 6600 50  0001 C CNN
+F 3 "" H 5750 6600 50  0001 C CNN
+	1    5750 6600
 	1    0    0    -1
 $EndComp
@@
 L power:GND #PWR?
 U 1 1 5E48745D
-P 5850 7200
-F 0 "#PWR?" H 5850 6950 50  0001 C CNN
-F 1 "GND" H 5855 7027 50  0000 C CNN
-F 2 "" H 5850 7200 50  0001 C CNN
-F 3 "" H 5850 7200 50  0001 C CNN
-	1    5850 7200
-	1    0    0    -1
-$EndComp
-Wire Wire Line
-	5550 6650 5700 6650
-Wire Wire Line
-	5700 6650 5700 6600
-Wire Wire Line
-	5550 6950 5850 6950
-Wire Wire Line
-	5850 6750 5850 6950
-Wire Wire Line
-	5550 6750 5850 6750
+P 5750 7200
+F 0 "#PWR?" H 5750 6950 50  0001 C CNN
+F 1 "GND" H 5755 7027 50  0000 C CNN
+F 2 "" H 5750 7200 50  0001 C CNN
+F 3 "" H 5750 7200 50  0001 C CNN
+	1    5750 7200
+	1    0    0    -1
+$EndComp
 Wire Wire Line
 	1850 1100 1850 1000
@@
 U 1 1 5E4E1068
 P 1300 1300
-F 0 "J?" H 1400 1800 50  0000 C CNN
-F 1 "USB_B" H 1400 1700 50  0000 C CNN
+F 0 "J?" H 1250 1800 50  0000 C CNN
+F 1 "USB_B" H 1300 1700 50  0000 C CNN
 F 2 "Connector_USB:USB_B_OST_USB-B1HSxx_Horizontal" H 1450 1250 50  0001 C CNN
 F 3 " ~" H 1450 1250 50  0001 C CNN
@@
 $EndComp
 Wire Wire Line
-	8700 1250 8550 1250
-Connection ~ 8700 1250
-Wire Wire Line
-	8700 1250 8700 1350
-Text GLabel 8550 1250 0    50   Input ~ 0
+	8700 1200 8550 1200
+Text GLabel 8550 1200 0    50   Input ~ 0
 RST
 Wire Wire Line
@@
 	1    0    0    -1
 $EndComp
-Wire Wire Line
-	5550 7150 5850 7150
-Wire Wire Line
-	5850 7150 5850 7200
-Wire Wire Line
-	5850 7150 5850 6950
-Connection ~ 5850 7150
-Connection ~ 5850 6950
 Wire Wire Line
 	9900 4150 10000 4150
@@
 	0    -1   -1   0
 $EndComp
+Wire Wire Line
+	8700 1150 8700 1200
+Connection ~ 8700 1200
+Wire Wire Line
+	8700 1200 8700 1350
+Wire Wire Line
+	5750 6750 5750 6950
+Wire Wire Line
+	5550 7150 5750 7150
+Connection ~ 5750 7150
+Wire Wire Line
+	5750 7150 5750 7200
+Wire Wire Line
+	5550 6950 5750 6950
+Connection ~ 5750 6950
+Wire Wire Line
+	5750 6950 5750 7150
+Wire Wire Line
+	5550 6750 5750 6750
+Wire Wire Line
+	5550 6650 5750 6650
+Wire Wire Line
+	5750 6650 5750 6600
 $EndSCHEMATC

Commit message: PCB build started
Parts:
- removed J?: Stepper, Connector_PinSocket_2.00mm:PinSocket_1x04_P2.00mm_Vertical, symbol Connector:Conn_01x04_Male
- removed J?: UART, symbol Connector:Conn_01x02_Male
- added J1: Stepper, Connector_PinHeader_2.54mm:PinHeader_1x06_P2.54mm_Vertical, symbol Connector:Conn_01x06_Male
- added J5: UART, Connector_PinHeader_2.54mm:PinHeader_1x02_P2.54mm_Vertical, symbol Connector:Conn_01x02_Male
- C1, C2, C3, C4: renamed from C?; footprint (none) -> Capacitor_SMD:C_0603_1608Metric
- D1, D2: renamed from D?; footprint Diode_SMD:D_0603_1608Metric_Pad1.05x0.95mm_HandSolder -> Diode_SMD:D_0603_1608Metric_Castellated
- J3: renamed from J?; footprint (none) -> Connector_PinHeader_2.54mm:PinHeader_1x02_P2.54mm_Vertical
- J4: renamed from J?; footprint Connector_JST:JST_PH_S2B-PH-K_1x02_P2.00mm_Horizontal -> Connector_PinHeader_2.54mm:PinHeader_1x02_P2.54mm_Vertical
- J6: renamed from J?; footprint (none) -> Connector_PinHeader_2.54mm:PinHeader_1x06_P2.54mm_Vertical
- J7: renamed from J?; footprint (none) -> Connector_PinHeader_2.54mm:PinHeader_2x03_P2.54mm_Vertical
- JP1, JP2, JP3: renamed from JP?; footprint (none) -> Jumper:SolderJumper-3_P1.3mm_Open_RoundedPad1.0x1.5mm_NumberLabels
- R1, R2, R3, R5, R6, R7: renamed from R?; footprint (none) -> Resistor_SMD:R_0603_1608Metric
- R4: renamed from R3; footprint (none) -> Resistor_SMD:R_0603_1608Metric
- Y1: renamed from Y?; footprint (none) -> Crystal:Crystal_SMD_3225-4Pin_3.2x2.5mm_HandSoldering
- gave numbers to parts that had none: 5
- renumbered C1 to C5
Connections:
- no-connect marks 18 -> 20
