File: motorboard/motorboard.sch (KiCad schematic (older format))
At the start: 29 parts, among them J1 Stepper, J2 USB_B, J3 DC Motor, J4 LiPo, J5 UART, J6 Encoders, J7 ICSP, U1 TB6612FNG, U2 ATmega32U4-AU, Y1 8MHz

Commit message: GitHub works again!
Parts:
- removed J2: USB_B, Connector_USB:USB_B_OST_USB-B1HSxx_Horizontal, symbol Connector:USB_B
- added J2: USB_B_Micro, symbol Connector:USB_B_Micro
Connections:
- net D+: now also J2.3 (D+)
- net D-: now also J2.2 (D-)
- net GND: now also J2.5 (GND), J2.6 (Shield)
- net VBUS: now also J2.1 (VBUS)
- no-connect marks 20 -> 21
Other:
- moved on the sheet: J4
Changed lines of the file:
@@
 $EndComp
 Wire Wire Line
-	1850 1100 1850 1000
-Wire Wire Line
-	1600 1100 1850 1100
-Text GLabel 1750 1400 2    50   Input ~ 0
+	1800 1100 1800 1000
+Wire Wire Line
+	1550 1100 1800 1100
+Text GLabel 1700 1400 2    50   Input ~ 0
 D-
-Text GLabel 1750 1300 2    50   Input ~ 0
+Text GLabel 1700 1300 2    50   Input ~ 0
 D+
 Wire Wire Line
-	1600 1400 1750 1400
-Wire Wire Line
-	1600 1300 1750 1300
-$Comp
-L Connector:USB_B J2
-U 1 1 5E4E1068
-P 1300 1300
-F 0 "J2" H 1250 1800 50  0000 C CNN
-F 1 "USB_B" H 1300 1700 50  0000 C CNN
-F 2 "Connector_USB:USB_B_OST_USB-B1HSxx_Horizontal" H 1450 1250 50  0001 C CNN
-F 3 " ~" H 1450 1250 50  0001 C CNN
-	1    1300 1300
-	1    0    0    -1
-$EndComp
-Connection ~ 1300 1750
-Wire Wire Line
-	1300 1750 1300 1700
-Wire Wire Line
-	1300 1750 1300 1800
-Wire Wire Line
-	1200 1750 1300 1750
-Wire Wire Line
-	1200 1700 1200 1750
+	1550 1400 1700 1400
+Wire Wire Line
+	1550 1300 1700 1300
+Connection ~ 1250 1750
+Wire Wire Line
+	1250 1750 1250 1700
+Wire Wire Line
+	1250 1750 1250 1800
+Wire Wire Line
+	1150 1750 1250 1750
+Wire Wire Line
+	1150 1700 1150 1750
 $Comp
 L power:GND #PWR03
 U 1 1 5E3E5F09
-P 1300 1800
-F 0 "#PWR03" H 1300 1550 50  0001 C CNN
-F 1 "GND" H 1350 1600 50  0000 C CNN
-F 2 "" H 1300 1800 50  0001 C CNN
-F 3 "" H 1300 1800 50  0001 C CNN
-	1    1300 1800
+P 1250 1800
+F 0 "#PWR03" H 1250 1550 50  0001 C CNN
+F 1 "GND" H 1300 1600 50  0000 C CNN
+F 2 "" H 1250 1800 50  0001 C CNN
+F 3 "" H 1250 1800 50  0001 C CNN
+	1    1250 1800
 	1    0    0    -1
 $EndComp
@@
 L power:VBUS #PWR04
 U 1 1 5E61CDDB
-P 1850 1000
-F 0 "#PWR04" H 1850 850 50  0001 C CNN
-F 1 "VBUS" H 1865 1173 50  0000 C CNN
-F 2 "" H 1850 1000 50  0001 C CNN
-F 3 "" H 1850 1000 50  0001 C CNN
-	1    1850 1000
-	1    0    0    -1
-$EndComp
-Wire Wire Line
-	2850 1550 2700 1550
-Wire Wire Line
-	2700 1450 2850 1450
+P 1800 1000
+F 0 "#PWR04" H 1800 850 50  0001 C CNN
+F 1 "VBUS" H 1815 1173 50  0000 C CNN
+F 2 "" H 1800 1000 50  0001 C CNN
+F 3 "" H 1800 1000 50  0001 C CNN
+	1    1800 1000
+	1    0    0    -1
+$EndComp
+Wire Wire Line
+	2850 1500 2700 1500
+Wire Wire Line
+	2700 1400 2850 1400
 $Comp
 L power:GND #PWR?
 U 1 1 5E649C1D
-P 2850 1600
+P 2850 1550
 AR Path="/5DAD2180/5E649C1D" Ref="#PWR?"  Part="1"
 AR Path="/5E649C1D" Ref="#PWR08"  Part="1"
-F 0 "#PWR08" H 2850 1350 50  0001 C CNN
-F 1 "GND" H 2855 1427 50  0000 C CNN
-F 2 "" H 2850 1600 50  0001 C CNN
-F 3 "" H 2850 1600 50  0001 C CNN
-	1    2850 1600
+F 0 "#PWR08" H 2850 1300 50  0001 C CNN
+F 1 "GND" H 2855 1377 50  0000 C CNN
+F 2 "" H 2850 1550 50  0001 C CNN
+F 3 "" H 2850 1550 50  0001 C CNN
+	1    2850 1550
 	1    0    0    -1
 $EndComp
@@
 L Connector_Generic:Conn_01x02 J?
 U 1 1 5E649C23
-P 2500 1450
+P 2500 1400
 AR Path="/5DAD2180/5E649C23" Ref="J?"  Part="1"
 AR Path="/5E649C23" Ref="J4"  Part="1"
-F 0 "J4" H 2418 1667 50  0000 C CNN
-F 1 "LiPo" H 2418 1576 50  0000 C CNN
-F 2 "Connector_PinHeader_2.54mm:PinHeader_1x02_P2.54mm_Vertical" H 2500 1450 50  0001 C CNN
-F 3 "~" H 2500 1450 50  0001 C CNN
-	1    2500 1450
+F 0 "J4" H 2418 1617 50  0000 C CNN
+F 1 "LiPo" H 2418 1526 50  0000 C CNN
+F 2 "Connector_PinHeader_2.54mm:PinHeader_1x02_P2.54mm_Vertical" H 2500 1400 50  0001 C CNN
+F 3 "~" H 2500 1400 50  0001 C CNN
+	1    2500 1400
 	-1   0    0    -1
 $EndComp
 Wire Wire Line
-	2850 1400 2850 1450
-Wire Wire Line
-	2850 1600 2850 1550
+	2850 1350 2850 1400
+Wire Wire Line
+	2850 1550 2850 1500
 $Comp
 L power:+15V #PWR?
 U 1 1 5E649C2B
-P 2850 1400
+P 2850 1350
 AR Path="/5DAD2180/5E649C2B" Ref="#PWR?"  Part="1"
 AR Path="/5E649C2B" Ref="#PWR07"  Part="1"
-F 0 "#PWR07" H 2850 1250 50  0001 C CNN
-F 1 "+15V" H 2865 1573 50  0000 C CNN
-F 2 "" H 2850 1400 50  0001 C CNN
-F 3 "" H 2850 1400 50  0001 C CNN
-	1    2850 1400
+F 0 "#PWR07" H 2850 1200 50  0001 C CNN
+F 1 "+15V" H 2865 1523 50  0000 C CNN
+F 2 "" H 2850 1350 50  0001 C CNN
+F 3 "" H 2850 1350 50  0001 C CNN
+	1    2850 1350
 	1    0    0    -1
 $EndComp
@@
 	1    0    0    -1
 $EndComp
+$Comp
+L Connector:USB_B_Micro J2
+U 1 1 5E58BFE0
+P 1250 1300
+F 0 "J2" H 1307 1767 50  0000 C CNN
+F 1 "USB_B_Micro" H 1307 1676 50  0000 C CNN
+F 2 "" H 1400 1250 50  0001 C CNN
+F 3 "~" H 1400 1250 50  0001 C CNN
+	1    1250 1300
+	1    0    0    -1
+$EndComp
+NoConn ~ 1550 1500
 $EndSCHEMATC

Commit message: It broke again
Parts:
- J2: footprint (none) -> Connector_USB:USB_Micro-B_Molex-105017-0001
Connections:
- net +10V is gone; now on net +15V: U1.13 (VM2), U1.14 (VM3), U1.24 (VM1)
Changed lines of the file:
@@
 Wire Wire Line
 	2300 3350 2400 3350
-$Comp
-L power:+10V #PWR?
-U 1 1 5E394AC0
-P 2400 3050
-AR Path="/5E41532A/5E394AC0" Ref="#PWR?"  Part="1"
-AR Path="/5E394AC0" Ref="#PWR05"  Part="1"
-F 0 "#PWR05" H 2400 2900 50  0001 C CNN
-F 1 "+10V" H 2415 3223 50  0000 C CNN
-F 2 "" H 2400 3050 50  0001 C CNN
-F 3 "" H 2400 3050 50  0001 C CNN
-	1    2400 3050
-	1    0    0    -1
-$EndComp
 Wire Wire Line
 	2400 3350 2400 3050
@@
 F 0 "J2" H 1307 1767 50  0000 C CNN
 F 1 "USB_B_Micro" H 1307 1676 50  0000 C CNN
-F 2 "" H 1400 1250 50  0001 C CNN
+F 2 "Connector_USB:USB_Micro-B_Molex-105017-0001" H 1400 1250 50  0001 C CNN
 F 3 "~" H 1400 1250 50  0001 C CNN
 	1    1250 1300
@@
 $EndComp
 NoConn ~ 1550 1500
+$Comp
+L power:+15V #PWR?
+U 1 1 5E52D87A
+P 2400 3050
+AR Path="/5DAD2180/5E52D87A" Ref="#PWR?"  Part="1"
+AR Path="/5E52D87A" Ref="#PWR?"  Part="1"
+F 0 "#PWR?" H 2400 2900 50  0001 C CNN
+F 1 "+15V" H 2415 3223 50  0000 C CNN
+F 2 "" H 2400 3050 50  0001 C CNN
+F 3 "" H 2400 3050 50  0001 C CNN
+	1    2400 3050
+	1    0    0    -1
+$EndComp
 $EndSCHEMATC

Commit message: ready for fab
Parts:
- C3, C4: value 33p -> 22p
- Y1: footprint Crystal:Crystal_SMD_3225-4Pin_3.2x2.5mm_HandSoldering -> Crystal:Crystal_HC18-U_Vertical
Changed lines of the file:
@@
 P 8200 1500
 F 0 "C3" V 8250 1400 50  0000 C CNN
-F 1 "33p" V 8050 1500 50  0000 C CNN
+F 1 "22p" V 8050 1500 50  0000 C CNN
 F 2 "Capacitor_SMD:C_0603_1608Metric" H 8200 1500 50  0001 C CNN
 F 3 "~" H 8200 1500 50  0001 C CNN
@@
 P 8200 1800
 F 0 "C4" V 8150 1700 50  0000 C CNN
-F 1 "33p" V 8300 1800 50  0000 C CNN
+F 1 "22p" V 8300 1800 50  0000 C CNN
 F 2 "Capacitor_SMD:C_0603_1608Metric" H 8200 1800 50  0001 C CNN
 F 3 "~" H 8200 1800 50  0001 C CNN
@@
 F 0 "Y1" V 8450 1500 50  0000 R CNN
 F 1 "8MHz" V 8650 1750 50  0000 R CNN
-F 2 "Crystal:Crystal_SMD_3225-4Pin_3.2x2.5mm_HandSoldering" H 8450 1650 50  0001 C CNN
+F 2 "Crystal:Crystal_HC18-U_Vertical" H 8450 1650 50  0001 C CNN
 F 3 "~" H 8450 1650 50  0001 C CNN
 	1    8450 1650
@@
 P 2400 3050
 AR Path="/5DAD2180/5E52D87A" Ref="#PWR?"  Part="1"
-AR Path="/5E52D87A" Ref="#PWR?"  Part="1"
-F 0 "#PWR?" H 2400 2900 50  0001 C CNN
+AR Path="/5E52D87A" Ref="#PWR0101"  Part="1"
+F 0 "#PWR0101" H 2400 2900 50  0001 C CNN
 F 1 "+15V" H 2415 3223 50  0000 C CNN
 F 2 "" H 2400 3050 50  0001 C CNN

Commit message: noob error fixed
Connections:
- net VBUS is gone; now on net +5V: J2.1 (VBUS)
Changed lines of the file:
@@
 	1800 1100 1800 1000
 Wire Wire Line
-	1550 1100 1800 1100
+	1550 1100 1650 1100
 Text GLabel 1700 1400 2    50   Input ~ 0
 D-
@@
 P 1800 1000
 F 0 "#PWR04" H 1800 850 50  0001 C CNN
-F 1 "VBUS" H 1815 1173 50  0000 C CNN
+F 1 "VBUS" H 1900 1150 50  0000 C CNN
 F 2 "" H 1800 1000 50  0001 C CNN
 F 3 "" H 1800 1000 50  0001 C CNN
@@
 	1    0    0    -1
 $EndComp
+$Comp
+L power:+5V #PWR0102
+U 1 1 5E744975
+P 1650 1000
+F 0 "#PWR0102" H 1650 850 50  0001 C CNN
+F 1 "+5V" H 1665 1173 50  0000 C CNN
+F 2 "" H 1650 1000 50  0001 C CNN
+F 3 "" H 1650 1000 50  0001 C CNN
+	1    1650 1000
+	1    0    0    -1
+$EndComp
+Wire Wire Line
+	1650 1000 1650 1100
+Connection ~ 1650 1100
+Wire Wire Line
+	1650 1100 1800 1100
 $EndSCHEMATC

Commit message: rev2 started
Parts:
- removed J4: LiPo, Connector_PinHeader_2.54mm:PinHeader_1x02_P2.54mm_Vertical, symbol Connector_Generic:Conn_01x02
- added J4: LiPo, xt30:AMASS_XT30PW-M_1x02_P2.50mm_Horizontal, symbol Connector:Conn_01x02_Male
Connections:
- net +15V: now also J4.1 (Pin_1)
- net DIR: now also U2.28 (PB4)
- net GND: now also J4.2 (Pin_2)
- net STEP: now also U2.29 (PB5)
- no-connect marks 21 -> 19
Changed lines of the file:
@@
 	1    0    0    -1
-$EndComp
-$Comp
-L Connector_Generic:Conn_01x02 J?
-U 1 1 5E649C23
-P 2500 1400
-AR Path="/5DAD2180/5E649C23" Ref="J?"  Part="1"
-AR Path="/5E649C23" Ref="J4"  Part="1"
-F 0 "J4" H 2418 1617 50  0000 C CNN
-F 1 "LiPo" H 2418 1526 50  0000 C CNN
-F 2 "Connector_PinHeader_2.54mm:PinHeader_1x02_P2.54mm_Vertical" H 2500 1400 50  0001 C CNN
-F 3 "~" H 2500 1400 50  0001 C CNN
-	1    2500 1400
-	-1   0    0    -1
 $EndComp
 Wire Wire Line
@@
 NoConn ~ 9900 3150
 NoConn ~ 9900 3050
-NoConn ~ 9900 1850
-NoConn ~ 9900 1750
 NoConn ~ 9900 1350
 Text GLabel 10000 4150 2    50   Input ~ 0
@@
 $EndComp
 $Comp
-L power:+5V #PWR?
+L power:+5V #PWR0102
 U 1 1 5E745145
 P 1650 1000
-F 0 "#PWR?" H 1650 850 50  0001 C CNN
+F 0 "#PWR0102" H 1650 850 50  0001 C CNN
 F 1 "+5V" H 1665 1173 50  0000 C CNN
 F 2 "" H 1650 1000 50  0001 C CNN
@@
 Wire Wire Line
 	1650 1100 1800 1100
+Text GLabel 10100 1750 2    50   Input ~ 0
+DIR
+Text GLabel 10100 1850 2    50   Input ~ 0
+STEP
+Wire Wire Line
+	10100 1750 9900 1750
+Wire Wire Line
+	10100 1850 9900 1850
+$Comp
+L Connector:Conn_01x02_Male J?
+U 1 1 5E807167
+P 2500 1400
+AR Path="/5DAD2180/5E807167" Ref="J?"  Part="1"
+AR Path="/5E807167" Ref="J4"  Part="1"
+F 0 "J4" H 2550 1500 50  0000 C CNN
+F 1 "LiPo" V 2400 1350 50  0000 C CNN
+F 2 "xt30:AMASS_XT30PW-M_1x02_P2.50mm_Horizontal" H 2500 1400 50  0001 C CNN
+F 3 "~" H 2500 1400 50  0001 C CNN
+	1    2500 1400
+	1    0    0    -1
+$EndComp
 $EndSCHEMATC

Commit message: 4 pin header for stepper
Parts:
- J1: symbol Connector:Conn_01x06_Male -> Connector:Conn_01x04_Male
- J4: footprint xt30:AMASS_XT30PW-M_1x02_P2.50mm_Horizontal -> xt30:AMASS_XT30UPB-F_1x02_P5.0mm_Vertical
- Y1: footprint Crystal:Crystal_HC18-U_Vertical -> Crystal:Crystal_HC49-4H_Vertical
Connections:
- net 1A: now also J1.2 (Pin_2); no longer J1.3 (Pin_3)
- net 2A: now also J1.3 (Pin_3); no longer J1.4 (Pin_4)
- net 2B: now also J1.4 (Pin_4); no longer J1.6 (Pin_6)
- no-connect marks 19 -> 18
Changed lines of the file:
@@
 	9300 4650 9300 4700
 Connection ~ 9300 4650
-Text GLabel 1650 6600 2    50   Input ~ 0
+Text GLabel 1600 6700 2    50   Input ~ 0
 1B
-Text GLabel 1650 6800 2    50   Input ~ 0
+Text GLabel 1600 6800 2    50   Input ~ 0
 1A
-Text GLabel 1650 6900 2    50   Input ~ 0
+Text GLabel 1600 6900 2    50   Input ~ 0
 2A
-Text GLabel 1650 7100 2    50   Input ~ 0
+Text GLabel 1600 7000 2    50   Input ~ 0
 2B
-Text Notes 1850 6650 0    50   ~ 0
+Text Notes 1800 6750 0    50   ~ 0
 Black
-Text Notes 1850 6850 0    50   ~ 0
+Text Notes 1800 6850 0    50   ~ 0
 Green
-Text Notes 1850 6950 0    50   ~ 0
+Text Notes 1800 6950 0    50   ~ 0
 Blue
-Text Notes 1850 7150 0    50   ~ 0
+Text Notes 1800 7050 0    50   ~ 0
 Red
 $Comp
@@
 F 0 "Y1" V 8450 1500 50  0000 R CNN
 F 1 "8MHz" V 8650 1750 50  0000 R CNN
-F 2 "Crystal:Crystal_HC18-U_Vertical" H 8450 1650 50  0001 C CNN
+F 2 "Crystal:Crystal_HC49-4H_Vertical" H 8450 1650 50  0001 C CNN
 F 3 "~" H 8450 1650 50  0001 C CNN
 	1    8450 1650
@@
 Wire Wire Line
 	5750 6650 5750 6600
-$Comp
-L Connector:Conn_01x06_Male J1
-U 1 1 5E510B96
-P 1300 6800
-F 0 "J1" H 1200 7200 50  0000 C CNN
-F 1 "Stepper" H 1250 7100 50  0000 C CNN
-F 2 "Connector_PinHeader_2.54mm:PinHeader_1x06_P2.54mm_Vertical" H 1300 6800 50  0001 C CNN
-F 3 "~" H 1300 6800 50  0001 C CNN
-	1    1300 6800
-	1    0    0    -1
-$EndComp
-Wire Wire Line
-	1500 7100 1650 7100
-Wire Wire Line
-	1500 6900 1650 6900
-Wire Wire Line
-	1500 6800 1650 6800
-Wire Wire Line
-	1500 6600 1650 6600
-NoConn ~ 1500 6700
-NoConn ~ 1500 7000
+Wire Wire Line
+	1450 7000 1600 7000
+Wire Wire Line
+	1450 6900 1600 6900
+Wire Wire Line
+	1450 6800 1600 6800
+Wire Wire Line
+	1450 6700 1600 6700
 $Comp
 L Connector:Conn_01x02_Male J5
@@
 F 0 "J4" H 2550 1500 50  0000 C CNN
 F 1 "LiPo" V 2400 1350 50  0000 C CNN
-F 2 "xt30:AMASS_XT30PW-M_1x02_P2.50mm_Horizontal" H 2500 1400 50  0001 C CNN
+F 2 "xt30:AMASS_XT30UPB-F_1x02_P5.0mm_Vertical" H 2500 1400 50  0001 C CNN
 F 3 "~" H 2500 1400 50  0001 C CNN
 	1    2500 1400
 	1    0    0    -1
 $EndComp
+$Comp
+L Connector:Conn_01x04_Male J1
+U 1 1 5E510B96
+P 1250 6800
+F 0 "J1" H 1050 7100 50  0000 C CNN
+F 1 "Stepper" H 1100 7000 50  0000 C CNN
+F 2 "Connector_PinHeader_2.54mm:PinHeader_1x06_P2.54mm_Vertical" H 1250 6800 50  0001 C CNN
+F 3 "~" H 1250 6800 50  0001 C CNN
+	1    1250 6800
+	1    0    0    -1
+$EndComp
+NoConn ~ 4500 2650
 $EndSCHEMATC

Commit message: edit
Parts:
- J1: footprint Connector_PinHeader_2.54mm:PinHeader_1x06_P2.54mm_Vertical -> Connector_PinHeader_2.54mm:PinHeader_1x04_P2.54mm_Vertical
Changed lines of the file:
@@
 F 0 "J1" H 1050 7100 50  0000 C CNN
 F 1 "Stepper" H 1100 7000 50  0000 C CNN
-F 2 "Connector_PinHeader_2.54mm:PinHeader_1x06_P2.54mm_Vertical" H 1250 6800 50  0001 C CNN
+F 2 "Connector_PinHeader_2.54mm:PinHeader_1x04_P2.54mm_Vertical" H 1250 6800 50  0001 C CNN
 F 3 "~" H 1250 6800 50  0001 C CNN
 	1    1250 6800
