File: motorboard/_autosave-motorboard.sch (KiCad schematic (older format))
At the start: 29 parts, among them J1 Stepper, J2 USB_B_Micro, J3 DC Motor, J4 LiPo, J5 UART, J6 Encoders, J7 ICSP, U1 TB6612FNG, U2 ATmega32U4-AU, Y1 8MHz

Commit message: It broke again
Parts:
- C3, C4: value 33p -> 22p
- Y1: footprint Crystal:Crystal_SMD_3225-4Pin_3.2x2.5mm_HandSoldering -> Crystal:Crystal_HC18-U_Vertical
Connections:
- net +10V is gone; now on net +15V: U1.13 (VM2), U1.14 (VM3), U1.24 (VM1)
Changed lines of the file:
@@
 Wire Wire Line
 	2300 3350 2400 3350
-$Comp
-L power:+10V #PWR?
-U 1 1 5E394AC0
-P 2400 3050
-AR Path="/5E41532A/5E394AC0" Ref="#PWR?"  Part="1"
-AR Path="/5E394AC0" Ref="#PWR05"  Part="1"
-F 0 "#PWR05" H 2400 2900 50  0001 C CNN
-F 1 "+10V" H 2415 3223 50  0000 C CNN
-F 2 "" H 2400 3050 50  0001 C CNN
-F 3 "" H 2400 3050 50  0001 C CNN
-	1    2400 3050
-	1    0    0    -1
-$EndComp
 Wire Wire Line
 	2400 3350 2400 3050
@@
 P 8200 1500
 F 0 "C3" V 8250 1400 50  0000 C CNN
-F 1 "33p" V 8050 1500 50  0000 C CNN
+F 1 "22p" V 8050 1500 50  0000 C CNN
 F 2 "Capacitor_SMD:C_0603_1608Metric" H 8200 1500 50  0001 C CNN
 F 3 "~" H 8200 1500 50  0001 C CNN
@@
 P 8200 1800
 F 0 "C4" V 8150 1700 50  0000 C CNN
-F 1 "33p" V 8300 1800 50  0000 C CNN
+F 1 "22p" V 8300 1800 50  0000 C CNN
 F 2 "Capacitor_SMD:C_0603_1608Metric" H 8200 1800 50  0001 C CNN
 F 3 "~" H 8200 1800 50  0001 C CNN
@@
 F 0 "Y1" V 8450 1500 50  0000 R CNN
 F 1 "8MHz" V 8650 1750 50  0000 R CNN
-F 2 "Crystal:Crystal_SMD_3225-4Pin_3.2x2.5mm_HandSoldering" H 8450 1650 50  0001 C CNN
+F 2 "Crystal:Crystal_HC18-U_Vertical" H 8450 1650 50  0001 C CNN
 F 3 "~" H 8450 1650 50  0001 C CNN
 	1    8450 1650
@@
 $EndComp
 NoConn ~ 1550 1500
+$Comp
+L power:+15V #PWR?
+U 1 1 5E52D87A
+P 2400 3050
+AR Path="/5DAD2180/5E52D87A" Ref="#PWR?"  Part="1"
+AR Path="/5E52D87A" Ref="#PWR0101"  Part="1"
+F 0 "#PWR0101" H 2400 2900 50  0001 C CNN
+F 1 "+15V" H 2415 3223 50  0000 C CNN
+F 2 "" H 2400 3050 50  0001 C CNN
+F 3 "" H 2400 3050 50  0001 C CNN
+	1    2400 3050
+	1    0    0    -1
+$EndComp
 $EndSCHEMATC
