File: motorboard/power.sch (KiCad schematic (older format))
At the start: 19 parts, among them J8 Separate LiPo, Q1 PMV20ENR, U3 TPS2412PW, U4 TPS63070

Commit message: rev2 started
Parts:
- removed J8: Separate LiPo, Connector_PinHeader_2.54mm:PinHeader_1x02_P2.54mm_Vertical, symbol Connector:Conn_01x02_Male
- added J8: Separate LiPo, Connector_PinHeader_2.54mm:PinHeader_1x02_P2.54mm_Vertical, symbol Connector_Generic:Conn_01x02
Connections:
- net GND: now also J8.2 (Pin_2)
- net at D4.2 (A): now also J8.1 (Pin_1)
Changed lines of the file:
@@
 Text Notes 4700 2150 0    303  ~ 61
 Powa!!
-$Comp
-L Connector:Conn_01x02_Male J8
-U 1 1 5E8D9BD5
-P 1800 5850
-F 0 "J8" H 1850 5950 50  0000 C CNN
-F 1 "Separate LiPo" V 1700 5800 50  0000 C CNN
-F 2 "Connector_PinHeader_2.54mm:PinHeader_1x02_P2.54mm_Vertical" H 1800 5850 50  0001 C CNN
-F 3 "~" H 1800 5850 50  0001 C CNN
-	1    1800 5850
-	1    0    0    -1
-$EndComp
 Wire Wire Line
 	2000 5950 2100 5950
@@
 Wire Wire Line
 	6250 4550 6250 4500
+$Comp
+L Connector_Generic:Conn_01x02 J8
+U 1 1 5E803995
+P 1800 5850
+AR Path="/5DAD2180/5E803995" Ref="J8"  Part="1"
+AR Path="/5E803995" Ref="J?"  Part="1"
+F 0 "J8" H 1800 6000 50  0000 C CNN
+F 1 "Separate LiPo" V 1950 5800 50  0000 C CNN
+F 2 "Connector_PinHeader_2.54mm:PinHeader_1x02_P2.54mm_Vertical" H 1800 5850 50  0001 C CNN
+F 3 "~" H 1800 5850 50  0001 C CNN
+	1    1800 5850
+	-1   0    0    -1
+$EndComp
 $EndSCHEMATC
